File: TESTPCB/charging-circuit/backups/20260414-191330/charging-circuit.kicad_pcb (KiCad board)
At the start: 2 copper layers, 82.6 x 94.6 mm, 270 parts, among them J1 2.54-1*6PHeader-RA, J10 Conn_01x02, J11 Conn_01x04, J2 USB_C_Receptacle_PowerOnly_6P, P1 Header-Male-2.54_2x2, P10 1.27mm/1*3p, P11 1.27mm/1*3p, P2 Header-Male-2.54_2x2, P3 1.27mm/1*3p, P4 1.27mm/1*3p, P5 1.27mm/1*3p, P6 1.27mm/1*3p, P7 1.27mm/1*3p, P8 1.27mm/1*3p, P9 1.27mm/1*3p, Q1 2N7002, Q10 AO3400A, Q11 AO3401A, Q2 CJQ4435, Q3 currentmirror, Q4 BSS84, Q5 AO4892, Q6 AO3401A, Q7 AO3401A, Q8 CJQ4435, Q9 AO3400A, SW1 TS-1088R-02026, U1 MAX17048G+T10, U10 BQ25606RGER, U11 Battery Input, U12 BQ24170RGYR, U13 TPS54302DDCR_C311983, U14 NTC10K/0805/F, U15 BQ76920PW, U16 NTC10K/0805/F, U17 HUSB238_002DD, U19 TPS54302DDCR_C311983, U2 MT3608, U20 TPS54302DDCR_C311983, U21 MCP73871, U22 SRP4020TA-1R0M, U3 MT3608, U4 TPL5110DDCT, U5 BQ25606RGER, U6 MT3608, U7 Z-21320110021001, U8 MAX3232CDBR, U9 ADS1115IDGSR

Commit message: Modularize charging-circuit schematic
Split the original flat KiCad schematic into hierarchical sheet files with a top-level overview.

Preserve PCB connectivity by restoring original component references and validating that the modular netlist matches the flat backup.

Include the modularization guide, sheet interfaces, and safety backups for the migrated design.
Connections:
- net 12BGND renamed /12BGND
- net 12BOOT renamed /12BOOT
- net 12BVOUT renamed /12BVOUT
- net 12BVSYS renamed /12BVSYS
- net 12FB renamed /12FB
- net 12GND renamed /12GND
- net 12VOUT renamed /12VOUT
- net 12VSYS renamed /12VSYS
- net 12V_Adapter renamed /12V_Adapter
- net 1D+ renamed /1D+
- net 1D- renamed /1D-
- net 2D+ renamed /2D+
- net 2D- renamed /2D-
- net 3V3BGND renamed /3V3BGND
- net 3V3BOOT renamed /3V3BOOT
- net 3V3BVOUT renamed /3V3BVOUT
- net 3V3BVSYS renamed /3V3BVSYS
- net 3V3FB renamed /3V3FB
- net 3V3GND renamed /3V3GND
- net 3V3VOUT renamed /3V3VOUT
- net 3V3VSYS renamed /3V3VSYS
- net 5BGND renamed /5BGND
- net 5BOOT renamed /5BOOT
- net 5BVOUT renamed /5BVOUT
- net 5BVSYS renamed /5BVSYS
- net 5FB renamed /5FB
- net 5GND renamed /5GND
- net 5VOUT renamed /5VOUT
- net 5VSYS renamed /5VSYS
- net A0 renamed /A0
- net A1 renamed /A1
- net A2 renamed /A2
- net A3 renamed /A3
- net ALERT-2-RASPI renamed /ALERT-2-RASPI
- net BAT2 renamed /BAT2
- net BAT_1 (+) renamed /BAT_1 (+)
- net BAT_1 (-) renamed /BAT_1 (-)
- net BAT_2 (-) renamed /BAT_2 (-)
- net BAT_3 (-) renamed /BAT_3 (-)
- net BTST renamed /BTST
- net CC1 renamed /CC1
- net CC2 renamed /CC2
- net CE2 renamed /CE2
- net CHG_GND renamed /CHG_GND
- net CHG_VBAT renamed /CHG_VBAT
- net D+ renamed /D+
- net D- renamed /D-
- net DSUB12V renamed /DSUB12V
- net DSUB3.3V renamed /DSUB3.3V
- net DSUBGND renamed /DSUBGND
- net FUELBAT renamed /FUELBAT
- net FUELGND renamed /FUELGND
- net FUELSCL renamed /FUELSCL
- net FUELSDA renamed /FUELSDA
- net GND1 renamed /GND1
- net GND2 renamed /GND2
- net ICHG2 renamed /ICHG2
- net ILIM2 renamed /ILIM2
- net ISET renamed /ISET
- net OTG2 renamed /OTG2
- net PACK- renamed /PACK-
- net PDGND renamed /PDGND
- net PDVOUT renamed /PDVOUT
- net PG2 renamed /PG2
- net PMID2 renamed /PMID2
- net PROTECT- renamed /PROTECT-
- net PWMSIG renamed /PWMSIG
- net REGN1 renamed /REGN1
- net REGN2 renamed /REGN2
- net RX renamed /RX
- net SCL-2-RASPI renamed /SCL-2-RASPI
- net SDA-2-RASPI renamed /SDA-2-RASPI
- net SLEEPGND renamed /SLEEPGND
- net SLEEPSIG renamed /SLEEPSIG
- net SLEEPVSYS renamed /SLEEPVSYS
- net STAT2 renamed /STAT2
- net SW2 renamed /SW2
- net SYS2 renamed /SYS2
- net TEMP12V renamed /TEMP12V
- net TEMPGND renamed /TEMPGND
- net TEMPSCL renamed /TEMPSCL
- net TEMPSDA renamed /TEMPSDA
- net TS2 renamed /TS2
- net TX renamed /TX
- net Temp3.3V renamed /Temp3.3V
- net UART_RX_13V renamed /UART_RX_13V
- net UART_TX_13V renamed /UART_TX_13V
- net USBGND renamed /USBGND
- net V1GND renamed /V1GND
- net V1VBAT renamed /V1VBAT
- net V1VBUS renamed /V1VBUS
- net V1VSYS renamed /V1VSYS
- net VAC2 renamed /VAC2
- net VBAT renamed /VBAT
- net VBAT1 renamed /VBAT1
- net VBUS renamed /VBUS
- net VBUS1 renamed /VBUS1
- net VBUS2 renamed /VBUS2
- net VC1 renamed /VC1
- net VCC renamed /VCC
- net VREF renamed /VREF
- net VSET renamed /VSET
- net VSET2 renamed /VSET2
- net VSYS1 renamed /VSYS1
- net base renamed /base
