File: vsens V3/charging-circuit/charging-circuit.kicad_pcb (KiCad board)
At the start: 2 copper layers, 82.6 x 94.6 mm, 270 parts, among them J1 2.54-1*6PHeader-RA, J10 Conn_01x02, J11 Conn_01x04, J2 USB_C_Receptacle_PowerOnly_6P, P1 Header-Male-2.54_2x2, P10 1.27mm/1*3p, P11 1.27mm/1*3p, P2 Header-Male-2.54_2x2, P3 1.27mm/1*3p, P4 1.27mm/1*3p, P5 1.27mm/1*3p, P6 1.27mm/1*3p, P7 1.27mm/1*3p, P8 1.27mm/1*3p, P9 1.27mm/1*3p, Q1 2N7002, Q10 AO3400A, Q11 AO3401A, Q2 CJQ4435, Q3 currentmirror, Q4 BSS84, Q5 AO4892, Q6 AO3401A, Q7 AO3401A, Q8 CJQ4435, Q9 AO3400A, SW1 TS-1088R-02026, U1 MAX17048G+T10, U10 BQ25606RGER, U11 Battery Input, U12 BQ24170RGYR, U13 TPS54302DDCR_C311983, U14 NTC10K/0805/F, U15 BQ76920PW, U16 NTC10K/0805/F, U17 HUSB238_002DD, U19 TPS54302DDCR_C311983, U2 MT3608, U20 TPS54302DDCR_C311983, U21 MCP73871, U22 SRP4020TA-1R0M, U3 MT3608, U4 TPL5110DDCT, U5 BQ25606RGER, U6 MT3608, U7 Z-21320110021001, U8 MAX3232CDBR, U9 ADS1115IDGSR

Commit message: Refactor code structure for improved readability and maintainability
Parts:
- removed ? (x38): , 
- removed the C1 at (40.6, 27.5)
- removed the C10 at (69.3, 32.3)
- removed C11, C40, C41, C46, C47: 22uF, PCM_JLCPCB:C_0603
- removed C13: 22uf, easyeda2kicad:C1206
- removed C14, C43, C50: 10uF, PCM_JLCPCB:C_0603
- removed the C15 at (55.8, 71.5)
- removed the C16 at (58.0, 73.0)
- removed the C2 at (40.6, 31.8)
- removed the C22 at (58.8, 75.5)
- removed the C29 at (46.7, 94.8)
- removed the C32 at (46.7, 93.3)
- removed the C33 at (56.7, 97.8)
- removed the C34 at (39.5, 100.2)
- removed the C35 at (33.5, 99.9)
- removed the C36 at (29.7, 99.2)
- removed the C37 at (39.7, 93.9)
- removed the C38 at (39.7, 95.4)
- removed C39: 47pF, PCM_JLCPCB:C_0603
- removed the C4 at (55.5, 28.6)
- removed C44, C45: 100nF, PCM_JLCPCB:C_0603
- removed C48: 75pf, easyeda2kicad:C0603
- removed C49: 100pF, PCM_JLCPCB:C_0603
- removed C51, C52: 4.7uF, PCM_JLCPCB:C_0603
- removed the C7 at (55.4, 32.3)
- removed the C9 at (52.3, 70.3)
- removed the D10 at (101.1, 48.1)
- removed D14: SS14, PCM_JLCPCB:D_SMA
- removed the D3 at (101.1, 50.3)
- removed the D4 at (33.6, 29.6)
- removed D5, D6: SS34, PCM_JLCPCB:D_SMA
- removed the D7 at (101.1, 52.6)
- removed the D8 at (52.8, 83.0)
- removed the D9 at (56.0, 83.8)
- removed the H2 at (40.3, 75.4)
- removed the H3 at (49.0, 77.0)
- removed the L1 at (51.8, 38.5)
- removed L2: 22uH, easyeda2kicad:IND-SMD_L7.5-W7.5
- removed the L3 at (65.6, 38.4)
- removed L5: 10uh, easyeda2kicad:IND-SMD_L7.5-W6.6
- removed L6: 6.8uh, easyeda2kicad:IND-SMD_L12.3-W12.3_SMDRI127
- removed L7: 15uh, easyeda2kicad:IND-SMD_L10.4-W10.3
- removed P10, P4, P5, P6, P7, P8, P9: 1.27mm/1*3p, easyeda2kicad:HDR-TH_3P-P1.27-V-M-1
- removed the P2 at (68.0, 77.7)
- removed the R1 at (39.0, 23.6)
- removed R10, R52: 22kΩ, PCM_JLCPCB:R_0603
- removed the R17 at (52.5, 80.0)
- removed the R18 at (66.5, 25.7)
- removed the R19 at (66.5, 24.0)
- removed the R2 at (37.9, 26.4)
- removed the R20 at (68.6, 24.9)
- removed the R22 at (57.8, 81.0)
- removed the R24 at (54.8, 81.0)
- removed the R25 at (56.3, 81.0)
- removed the R27 at (61.0, 76.3)
- removed the R28 at (60.5, 78.8)
- removed the R29 at (59.3, 81.0)
- removed the R30 at (37.3, 80.9)
- removed the R31 at (37.5, 75.9)
- removed R34: 330kΩ, PCM_JLCPCB:R_0603
- removed R37, R44, R49: 49.9kΩ, PCM_JLCPCB:R_0603
- removed R38, R45, R50: 100kΩ, PCM_JLCPCB:R_0603
- removed R39, RPROG3: 10kΩ, PCM_JLCPCB:R_0603
- removed R40, R42, R47: 511k, easyeda2kicad:R0805
- removed R41, R43, R48: 105k, easyeda2kicad:R0603
- removed R46: 3kΩ, PCM_JLCPCB:R_0603
- removed R51: 13.3k, easyeda2kicad:R0805
- removed R53: 2.2kΩ, PCM_JLCPCB:R_0603
- removed R56, R57, R58: 470Ω, PCM_JLCPCB:R_0603
- removed R59: 110kΩ, PCM_JLCPCB:R_0603
- removed the RPROG2 at (99.4, 57.8)
- removed the U10 at (54.5, 75.8)
- removed the U11 at (33.9, 69.7)
- removed U13, U19, U20: TPS54302DDCR_C311983, easyeda2kicad:SOT-23-6_L2.9-W1.6-P0.95-LS2.8-BL
- removed the U2 at (52.0, 29.9)
- removed U21: MCP73871, easyeda2kicad:QFN-20_L4.0-W4.0-P0.5-BL-EP
- removed U22: SRP4020TA-1R0M, easyeda2kicad:IND-SMD_L4.5-W4.1_SRP4020TA
- removed the U3 at (37.4, 30.4)
- removed U6: MT3608, PCM_JLCPCB:SOT-23-6_L2.9-W1.6-P0.95-LS2.8-BL
- removed USBC1: TYPE-C-31-M-12, easyeda2kicad:USB-C_SMD-TYPE-C-31-M-12_1
- added C1: 100uF, Capacitor_SMD:CP_Elec_8x10, F.Cu at (181.2, 85.7)
- added C1: 100uF, Capacitor_SMD:CP_Elec_8x10, F.Cu at (183.2, 108.8)
- added C2: 100nF, Capacitor_SMD:C_0603_1608Metric, F.Cu at (184.2, 92.2)
- added C2: 100nF, Capacitor_SMD:C_0603_1608Metric, F.Cu at (191.0, 123.5)
- added C3: 220uF, Capacitor_SMD:CP_Elec_8x10, F.Cu at (183.2, 118.6)
- added C3: 220uF, Capacitor_SMD:CP_Elec_8x10, F.Cu at (215.2, 85.5)
- added C4: 100nF, Capacitor_SMD:C_0603_1608Metric, F.Cu at (191.0, 126.0)
- added C4: 100nF, Capacitor_SMD:C_0603_1608Metric, F.Cu at (199.2, 79.8)
- added D1: SS34, Diode_SMD:D_SMA, F.Cu at (181.2, 125.8)
- added D1: LED, LED_SMD:LED_0603_1608Metric, F.Cu at (215.1, 77.0)
- added D2: LED, LED_SMD:LED_0603_1608Metric, F.Cu at (179.2, 129.4)
- added D2: SS34, Diode_SMD:D_SMA, F.Cu at (190.6, 93.8)
- added G***: LOGO, Logos:ampnics_full_10x10mm.kicad_sym, F.Cu at (182.5, 79.0)
- added J1: Conn_01x01_Pin, Connector_PinHeader_2.54mm:PinHeader_1x01_P2.54mm_Vertical, F.Cu at (178.1, 76.3)
- added J1: Conn_01x01_Pin, Connector_PinHeader_2.54mm:PinHeader_1x01_P2.54mm_Vertical, F.Cu at (191.3, 106.2)
- added J2: Conn_01x01_Pin, Connector_PinHeader_2.54mm:PinHeader_1x01_P2.54mm_Vertical, F.Cu at (178.1, 94.5)
- added J2: Conn_01x01_Pin, Connector_PinHeader_2.54mm:PinHeader_1x01_P2.54mm_Vertical, F.Cu at (191.3, 110.7)
- added J3: Conn_01x01_Pin, Connector_PinHeader_2.54mm:PinHeader_1x01_P2.54mm_Vertical, F.Cu at (218.3, 76.3)
- added J3: Conn_01x01_Pin, Connector_PinHeader_2.54mm:PinHeader_1x01_P2.54mm_Vertical, F.Cu at (191.3, 115.3)
- added J4: Conn_01x01_Pin, Connector_PinHeader_2.54mm:PinHeader_1x01_P2.54mm_Vertical, F.Cu at (218.3, 94.5)
- added J4: Conn_01x01_Pin, Connector_PinHeader_2.54mm:PinHeader_1x01_P2.54mm_Vertical, F.Cu at (191.3, 119.9)
- added L1: 47uH, Inductor_SMD:L_Bourns_SRR1208_12.7x12.7mm, F.Cu at (201.4, 123.0)
- added L1: 47uH, Inductor_SMD:L_Bourns_SRR1208_12.7x12.7mm, F.Cu at (204.0, 88.5)
- added R1: 4K7, Resistor_SMD:R_0603_1608Metric, F.Cu at (191.0, 128.5)
- added R1: 4K7, Resistor_SMD:R_0603_1608Metric, F.Cu at (213.2, 77.0)
- added RV1: 10K, Potentiometer_THT:Potentiometer_Bourns_3296W_Vertical, F.Cu at (209.4, 77.7)
- R3: value 3kΩ -> 1K; footprint PCM_JLCPCB:R_0603 -> Resistor_SMD:R_0603_1608Metric
- U1: value MAX17048G+T10 -> LM2596SX-5.0/NOPB; footprint easyeda2kicad:TDFN-8_L2.0-W2.0-P0.50-BL-EP1.2 -> easyeda2kicad:TO-263-5_L10.2-W8.9-P1.70-TL
- moved R3 155.3 mm to (199.2, 76.6), turned to -90 degrees
- moved U1 123.2 mm to (191.4, 84.2), turned to 90 degrees
- renumbered C26 to C10, C42 to C15, C53 to C16, C61 to C17, C5 to C18, C6 to C19, C72 to C20, C55 to C21, C56 to C22, C57 to C23, C54 to C24, C59 to C25, C58 to C26, C30 to C27, C31 to C28, C8 to C29, C23 to C30, C70 to C31, C71 to C32, C12 to C33, C20 to C34, C18 to C35, C21 to C36, C17 to C37, C19 to C38, C3 to C5, C27 to C6, C28 to C7, C25 to C8, C24 to C9, Cc0 to Cc2, D19 to D10, D1 to D11, D2 to D3, D11 to D4, D100 to D7, D12 to D8, D13 to D9, H6 to H1, H7 to H2, H5 to H3, H8 to H4, H9 to H5, H4 to H6, H11 to H7, J1 to J12, J2 to J5, L8 to L3, P3 to P1, P11 to P2, P1 to P3, Q8 to Q1, Q2 to Q10, Q3 to Q11, Q7 to Q2, Q6 to Q3, Q9 to Q4, Q10 to Q5, Q11 to Q6, Q5 to Q7, Q4 to Q8, Q1 to Q9, R4 to R11, R60 to R12, R61 to R13, R5 to R14, R62 to R15, R63 to R16, R6 to R17, R66 to R18, R64 to R19, R54 to R2, R7 to R20, R75 to R21, R76 to R22, R65 to R23, R11 to R24, R15 to R25, R16 to R26, R26 to R27, R32 to R28, R14 to R29, R8 to R3, R13 to R30, R21 to R31, R12 to R32, R55 to R33, R9 to R4, R33 to R5, R36 to R6, R77 to R7, R35 to R8, RPROG5 to RPROG2, R_AC2 to R_AC1, R_AC1 to R_AC2, Rc3 to Rc1, Rc1 to Rc3, Rc0 to Rc4, U15 to U10, U9 to U11, U8 to U12, U4 to U2, U7 to U3, U5 to U4, U17 to U5, U16 to U7, U12 to U8, U14 to U9
Connections:
- R3 pad 2: 5GND -> GND
- U1 pad 1: FUELGND -> LM2596_5V_VIN
- U1 pad 2: FUELBAT -> /LM2596 5V Buck/SW
- U1 pad 3: FUELBAT -> LM2596_5V_GND
- U1 pad 4: FUELGND -> LM2596_5V_VOUT
- U1 pad 5: FUELGND -> LM2596_5V_GND
- U1 pad 6: FUELGND -> LM2596_5V_GND
Routing:
- net GND1: track 64.8 -> 0.00 mm, vias 3 -> 0
- net VSYS1: track 46.1 -> 0.00 mm, vias 1 -> 0
- net V1GND: track 38.1 -> 0.00 mm, vias 1 -> 0
- net USBGND: track 37.6 -> 0.00 mm
- net 12BGND: track 36.7 -> 0.00 mm, vias 3 -> 0
- net 5BGND: track 30.2 -> 0.00 mm, vias 2 -> 0
- net V1VBUS: track 25.7 -> 0.00 mm, vias 3 -> 0
- net 3V3VSYS: track 23.2 -> 0.00 mm, vias 3 -> 0
- net 3V3GND: track 23.1 -> 0.00 mm
- net 5VSYS: track 22.9 -> 0.00 mm, vias 3 -> 0
- net 12GND: track 22.4 -> 0.00 mm, vias 2 -> 0
- net 12VSYS: track 21.9 -> 0.00 mm, vias 2 -> 0
- net 3V3BGND: track 21.8 -> 0.00 mm, vias 3 -> 0
- net 5GND: track 20.7 -> 0.00 mm
- net V1VSYS: track 20.6 -> 0.00 mm, vias 2 -> 0
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- added copper zone on F.Cu, net /SW
- added copper zone on F.Cu, net /VIN
- added copper zone on F.Cu, net /VOUT
- added copper zone on B.Cu, net GND
- added copper zone on F.Cu, net GND
- removed copper zone on F.Cu, net 12GND
- removed copper zone on F.Cu, net 3V3GND
- removed copper zone on F.Cu, net 5GND
Other:
- board size 82.6 x 94.6 mm -> 192.5 x 94.6 mm
- board text added: "${REFERENCE}"
- board text added: "+"
- board text added: "-"
- board text added: "BUCK CONVERTER NOV 25|v0.1.0 AMPNICS"
- board text added: "VIN"
- board text removed: "3V3"
- board text removed: "5V"
- board text removed: "VBAT"
