File: vsens V3/charging-circuit/charging-circuit.kicad_sch (KiCad schematic)
At the start: 0 parts

Commit message: Refactor code structure for improved readability and maintainability
Other:
- removed sheet 12BUCK
- removed sheet 12VLDO
- removed sheet 3.3BUCK
- removed sheet 3.3VLDO
- removed sheet 5BUCK
- removed sheet 5VLDO
- removed sheet CHARGE1
- removed sheet FUELGAUGE
- removed sheet LM2596 BUCK
- removed sheet USB+BAT
- removed sheet V1 IC
