File: vsens V3/charging-circuit/sheets/04_sleepmosfet.kicad_sch (KiCad schematic)
At the start: 8 parts, among them P3 1.27mm/1*3p, Q8 CJQ4435, U4 TPL5110DDCT

Commit message: Refactor code structure for improved readability and maintainability
Parts:
- renumbered C3 to C5, P3 to P1, Q8 to Q1, R54 to R2, R8 to R3, R9 to R4, U4 to U2
Changed lines of the file:
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@@
 		(dnp no)
 		(fields_autoplaced yes)
-		(property "Reference" "R9"
+		(property "Reference" "R4"
 			(at 179.07 113.0299 0)
 			(effects
@@
 			(project "charging-circuit"
 				(path "/529bc8a5-ffae-43ac-972d-caccc3afab85/46234f0e-61f2-45bf-9df2-e52d6b9d2e9e"
-					(reference "R9")
+					(reference "R4")
 					(unit 1)
 				)
@@
 		(dnp no)
 		(fields_autoplaced yes)
-		(property "Reference" "P3"
+		(property "Reference" "P1"
 			(at 100.33 80.01 0)
 			(effects
@@
 			(project "charging-circuit"
 				(path "/529bc8a5-ffae-43ac-972d-caccc3afab85/46234f0e-61f2-45bf-9df2-e52d6b9d2e9e"
-					(reference "P3")
+					(reference "P1")
 					(unit 1)
 				)
@@
 		(on_board yes)
 		(dnp no)
-		(property "Reference" "U4"
+		(property "Reference" "U2"
 			(at 135.636 99.822 0)
 			(effects
@@
 			(project "charging-circuit"
 				(path "/529bc8a5-ffae-43ac-972d-caccc3afab85/46234f0e-61f2-45bf-9df2-e52d6b9d2e9e"
-					(reference "U4")
+					(reference "U2")
 					(unit 1)
 				)
@@
 		(dnp no)
 		(fields_autoplaced yes)
-		(property "Reference" "R8"
+		(property "Reference" "R3"
 			(at 165.1 115.5699 0)
 			(effects
@@
 			(project "charging-circuit"
 				(path "/529bc8a5-ffae-43ac-972d-caccc3afab85/46234f0e-61f2-45bf-9df2-e52d6b9d2e9e"
-					(reference "R8")
+					(reference "R3")
 					(unit 1)
 				)
@@
 		(dnp no)
 		(fields_autoplaced yes)
-		(property "Reference" "C3"
+		(property "Reference" "C5"
 			(at 170.18 113.0299 0)
 			(effects
@@
 			(project "charging-circuit"
 				(path "/529bc8a5-ffae-43ac-972d-caccc3afab85/46234f0e-61f2-45bf-9df2-e52d6b9d2e9e"
-					(reference "C3")
+					(reference "C5")
 					(unit 1)
 				)
@@
 		(on_board yes)
 		(dnp no)
-		(property "Reference" "Q8"
+		(property "Reference" "Q1"
 			(at 178.816 111.76 0)
 			(effects
@@
 			(project "charging-circuit"
 				(path "/529bc8a5-ffae-43ac-972d-caccc3afab85/46234f0e-61f2-45bf-9df2-e52d6b9d2e9e"
-					(reference "Q8")
+					(reference "Q1")
 					(unit 1)
 				)
@@
 		(dnp no)
 		(fields_autoplaced yes)
-		(property "Reference" "R54"
+		(property "Reference" "R2"
 			(at 129.54 115.3199 90)
 			(effects
@@
 			(project "charging-circuit"
 				(path "/529bc8a5-ffae-43ac-972d-caccc3afab85/46234f0e-61f2-45bf-9df2-e52d6b9d2e9e"
-					(reference "R54")
-					(unit 1)
-				)
+					(reference "R2")
+					(unit 1)
+				)
