File: vsens V3/charging-circuit/sheets/07_ic2_breakout.kicad_sch (KiCad schematic)
At the start: 2 parts, among them U5 BQ25606RGER, U7 Z-21320110021001

Commit message: Refactor code structure for improved readability and maintainability
Parts:
- renumbered U7 to U3, U5 to U4
Changed lines of the file:
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@@
 		(dnp no)
 		(fields_autoplaced yes)
-		(property "Reference" "U5"
+		(property "Reference" "U4"
 			(at 115.57 60.96 0)
 			(effects
@@
 			(project "charging-circuit"
 				(path "/529bc8a5-ffae-43ac-972d-caccc3afab85/18b9eebe-215b-4696-a0de-5832208702d9"
-					(reference "U5")
+					(reference "U4")
 					(unit 1)
 				)
@@
 		(dnp no)
 		(fields_autoplaced yes)
-		(property "Reference" "U7"
+		(property "Reference" "U3"
 			(at 77.47 66.04 0)
 			(effects
@@
 			(project "charging-circuit"
 				(path "/529bc8a5-ffae-43ac-972d-caccc3afab85/18b9eebe-215b-4696-a0de-5832208702d9"
-					(reference "U7")
+					(reference "U3")
 					(unit 1)
 				)
