File: vsens V3/charging-circuit/sheets/14_3s_ic.kicad_sch (KiCad schematic)
At the start: 40 parts, among them P11 1.27mm/1*3p, Q10 AO3400A, Q11 AO3401A, Q9 AO3400A, U12 BQ24170RGYR, U16 NTC10K/0805/F

Commit message: Refactor code structure for improved readability and maintainability
Parts:
- renumbered C42 to C15, C53 to C16, C61 to C17, C5 to C18, C6 to C19, C72 to C20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
