File: vsens V3/charging-circuit/sheets/16_temp_heater.kicad_sch (KiCad schematic)
At the start: 13 parts, among them J1 2.54-1*6PHeader-RA, Q1 2N7002, Q2 CJQ4435, Q3 currentmirror, U9 ADS1115IDGSR

Commit message: Refactor code structure for improved readability and maintainability
Parts:
- renumbered C12 to C33, H4 to H6, J1 to J12, Q2 to Q10, Q3 to Q11, Q1 to Q9, R14 to R29, R13 to R30, R21 to R31, R12 to R32, R55 to R33, RPROG5 to RPROG2, U9 to U11
Changed lines of the file:
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@@
 		(on_board yes)
 		(dnp no)
-		(property "Reference" "R13"
+		(property "Reference" "R30"
 			(at 107.188 128.524 90)
 			(effects
@@
 			(project "charging-circuit"
 				(path "/529bc8a5-ffae-43ac-972d-caccc3afab85/c2b703a4-2e88-4383-8b77-8614951a81a3"
-					(reference "R13")
+					(reference "R30")
 					(unit 1)
 				)
@@
 		(dnp no)
 		(fields_autoplaced yes)
-		(property "Reference" "U9"
+		(property "Reference" "U11"
 			(at 133.35 116.84 0)
 			(effects
@@
 			(project "charging-circuit"
 				(path "/529bc8a5-ffae-43ac-972d-caccc3afab85/c2b703a4-2e88-4383-8b77-8614951a81a3"
-					(reference "U9")
+					(reference "U11")
 					(unit 1)
 				)
@@
 		(on_board yes)
 		(dnp no)
-		(property "Reference" "C12"
+		(property "Reference" "C33"
 			(at 167.386 135.382 90)
 			(effects
@@
 			(project "charging-circuit"
 				(path "/529bc8a5-ffae-43ac-972d-caccc3afab85/c2b703a4-2e88-4383-8b77-8614951a81a3"
-					(reference "C12")
+					(reference "C33")
 					(unit 1)
 				)
@@
 		(dnp no)
 		(fields_autoplaced yes)
-		(property "Reference" "RPROG5"
+		(property "Reference" "RPROG2"
 			(at 120.65 67.3099 0)
 			(effects
@@
 			(project "charging-circuit"
 				(path "/529bc8a5-ffae-43ac-972d-caccc3afab85/c2b703a4-2e88-4383-8b77-8614951a81a3"
-					(reference "RPROG5")
+					(reference "RPROG2")
 					(unit 1)
 				)
@@
 		(dnp no)
 		(fields_autoplaced yes)
-		(property "Reference" "Q1"
+		(property "Reference" "Q9"
 			(at 99.06 86.36 90)
 			(effects
@@
 			(project "charging-circuit"
 				(path "/529bc8a5-ffae-43ac-972d-caccc3afab85/c2b703a4-2e88-4383-8b77-8614951a81a3"
-					(reference "Q1")
+					(reference "Q9")
 					(unit 1)
 				)
@@
 		(on_board yes)
 		(dnp no)
-		(property "Reference" "R12"
+		(property "Reference" "R32"
 			(at 166.37 122.428 90)
 			(effects
@@
 			(project "charging-circuit"
 				(path "/529bc8a5-ffae-43ac-972d-caccc3afab85/c2b703a4-2e88-4383-8b77-8614951a81a3"
-					(reference "R12")
+					(reference "R32")
 					(unit 1)
 				)
@@
 		(dnp no)
 		(fields_autoplaced yes)
-		(property "Reference" "R55"
+		(property "Reference" "R33"
 			(at 176.53 85.09 90)
 			(effects
@@
 			(project "charging-circuit"
 				(path "/529bc8a5-ffae-43ac-972d-caccc3afab85/c2b703a4-2e88-4383-8b77-8614951a81a3"
-					(reference "R55")
+					(reference "R33")
 					(unit 1)
 				)
@@
 		(dnp no)
 		(fields_autoplaced yes)
-		(property "Reference" "J1"
+		(property "Reference" "J12"
 			(at 148.59 72.6449 0)
 			(effects
@@
 			(project "charging-circuit"
 				(path "/529bc8a5-ffae-43ac-972d-caccc3afab85/c2b703a4-2e88-4383-8b77-8614951a81a3"
-					(reference "J1")
+					(reference "J12")
 					(unit 1)
 				)
@@
 		(on_board yes)
 		(dnp no)
-		(property "Reference" "Q2"
+		(property "Reference" "Q10"
 			(at 110.744 73.406 0)
 			(effects
@@
 			(project "charging-circuit"
 				(path "/529bc8a5-ffae-43ac-972d-caccc3afab85/c2b703a4-2e88-4383-8b77-8614951a81a3"
-					(reference "Q2")
+					(reference "Q10")
 					(unit 1)
 				)
@@
 		(on_board yes)
 		(dnp no)
-		(property "Reference" "Q3"
+		(property "Reference" "Q11"
 			(at 160.0201 104.14 0)
 			(effects
@@
 			(project "charging-circuit"
 				(path "/529bc8a5-ffae-43ac-972d-caccc3afab85/c2b703a4-2e88-4383-8b77-8614951a81a3"
-					(reference "Q3")
+					(reference "Q11")
 					(unit 1)
 				)
@@
 		(dnp no)
 		(fields_autoplaced yes)
-		(property "Reference" "R21"
+		(property "Reference" "R31"
 			(at 165.1 130.81 90)
 			(effects
@@
 			(project "charging-circuit"
 				(path "/529bc8a5-ffae-43ac-972d-caccc3afab85/c2b703a4-2e88-4383-8b77-8614951a81a3"
-					(reference "R21")
+					(reference "R31")
 					(unit 1)
 				)
@@
 		(dnp no)
 		(fields_autoplaced yes)
-		(property "Reference" "R14"
+		(property "Reference" "R29"
 			(at 110.49 83.8199 0)
 			(effects
@@
 			(project "charging-circuit"
 				(path "/529bc8a5-ffae-43ac-972d-caccc3afab85/c2b703a4-2e88-4383-8b77-8614951a81a3"
-					(reference "R14")
+					(reference "R29")
 					(unit 1)
 				)
@@
 		(dnp no)
 		(fields_autoplaced yes)
-		(property "Reference" "H4"
+		(property "Reference" "H6"
 			(at 77.47 106.68 0)
 			(effects
@@
 			(project "charging-circuit"
 				(path "/529bc8a5-ffae-43ac-972d-caccc3afab85/c2b703a4-2e88-4383-8b77-8614951a81a3"
-					(reference "H4")
-					(unit 1)
-				)
+					(reference "H6")
+					(unit 1)
+				)
