File: vsens V3/charging-circuit/sheets/17_dsub_rs232.kicad_sch (KiCad schematic)
At the start: 8 parts, among them P1 Header-Male-2.54_2x2, U8 MAX3232CDBR

Commit message: Refactor code structure for improved readability and maintainability
Parts:
- renumbered C20 to C34, C18 to C35, C21 to C36, C17 to C37, C19 to C38, H11 to H7, P1 to P3, U8 to U12
Changed lines of the file:
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@@
 		(on_board yes)
 		(dnp no)
-		(property "Reference" "C17"
+		(property "Reference" "C37"
 			(at 121.666 89.662 90)
 			(effects
@@
 			(project "charging-circuit"
 				(path "/529bc8a5-ffae-43ac-972d-caccc3afab85/cebc8927-3eb9-4228-bd64-eb01f991daf3"
-					(reference "C17")
+					(reference "C37")
 					(unit 1)
 				)
@@
 		(on_board yes)
 		(dnp no)
-		(property "Reference" "C19"
+		(property "Reference" "C38"
 			(at 122.428 86.106 90)
 			(effects
@@
 			(project "charging-circuit"
 				(path "/529bc8a5-ffae-43ac-972d-caccc3afab85/cebc8927-3eb9-4228-bd64-eb01f991daf3"
-					(reference "C19")
+					(reference "C38")
 					(unit 1)
 				)
@@
 		(dnp no)
 		(fields_autoplaced yes)
-		(property "Reference" "H11"
+		(property "Reference" "H7"
 			(at 139.7 63.5 0)
 			(effects
@@
 			(project "charging-circuit"
 				(path "/529bc8a5-ffae-43ac-972d-caccc3afab85/cebc8927-3eb9-4228-bd64-eb01f991daf3"
-					(reference "H11")
+					(reference "H7")
 					(unit 1)
 				)
@@
 		(on_board yes)
 		(dnp no)
-		(property "Reference" "C20"
+		(property "Reference" "C34"
 			(at 76.708 87.376 90)
 			(effects
@@
 			(project "charging-circuit"
 				(path "/529bc8a5-ffae-43ac-972d-caccc3afab85/cebc8927-3eb9-4228-bd64-eb01f991daf3"
-					(reference "C20")
+					(reference "C34")
 					(unit 1)
 				)
@@
 		(on_board yes)
 		(dnp no)
-		(property "Reference" "C18"
+		(property "Reference" "C35"
 			(at 71.374 95.758 90)
 			(effects
@@
 			(project "charging-circuit"
 				(path "/529bc8a5-ffae-43ac-972d-caccc3afab85/cebc8927-3eb9-4228-bd64-eb01f991daf3"
-					(reference "C18")
+					(reference "C35")
 					(unit 1)
 				)
@@
 		(dnp no)
 		(fields_autoplaced yes)
-		(property "Reference" "U8"
+		(property "Reference" "U12"
 			(at 96.52 59.69 0)
 			(effects
@@
 			(project "charging-circuit"
 				(path "/529bc8a5-ffae-43ac-972d-caccc3afab85/cebc8927-3eb9-4228-bd64-eb01f991daf3"
-					(reference "U8")
+					(reference "U12")
 					(unit 1)
 				)
@@
 		(on_board yes)
 		(dnp no)
-		(property "Reference" "C21"
+		(property "Reference" "C36"
 			(at 81.788 110.236 90)
 			(effects
@@
 			(project "charging-circuit"
 				(path "/529bc8a5-ffae-43ac-972d-caccc3afab85/cebc8927-3eb9-4228-bd64-eb01f991daf3"
-					(reference "C21")
+					(reference "C36")
 					(unit 1)
 				)
@@
 		(dnp no)
 		(fields_autoplaced yes)
-		(property "Reference" "P1"
+		(property "Reference" "P3"
 			(at 135.89 105.41 0)
 			(effects
@@
 			(project "charging-circuit"
 				(path "/529bc8a5-ffae-43ac-972d-caccc3afab85/cebc8927-3eb9-4228-bd64-eb01f991daf3"
-					(reference "P1")
-					(unit 1)
-				)
+					(reference "P3")
+					(unit 1)
+				)
