File: vsens V3/charging-circuit/sheets/18_lm2596_adj_buck.kicad_sch (KiCad schematic)
At the start: 15 parts, among them J20 Conn_01x01_Pin, J21 Conn_01x01_Pin, J22 Conn_01x01_Pin, J23 Conn_01x01_Pin, U30 LM2596S-ADJ

Commit message: Refactor code structure for improved readability and maintainability
Parts:
- removed C902: 220uF, Capacitor_SMD:CP_Elec_8x10, symbol Device:C_Polarized
- removed D200: LED, LED_SMD:LED_0603_1608Metric, symbol Device:LED
- removed D201: SS34, Diode_SMD:D_SMA, symbol Diode:SS34
- removed J20, J21, J22, J23: Conn_01x01_Pin, Connector_PinHeader_2.54mm:PinHeader_1x01_P2.54mm_Vertical, symbol Connector:Conn_01x01_Pin
- removed U30: LM2596S-ADJ, Package_TO_SOT_SMD:TO-263-5_TabPin3, symbol Regulator_Switching:LM2596S-ADJ
- added C13: 220uF, Capacitor_SMD:CP_Elec_8x10, symbol Device:C_Polarized
- added D5: SS34, Diode_SMD:D_SMA, symbol Diode:SS34
- added D6: LED, LED_SMD:LED_0603_1608Metric, symbol Device:LED
- added J6, J7, J8, J9: Conn_01x01_Pin, Connector_PinHeader_2.54mm:PinHeader_1x01_P2.54mm_Vertical, symbol Connector:Conn_01x01_Pin
- added U6: LM2596SX-5.0/NOPB, easyeda2kicad:TO-263-5_L10.2-W8.9-P1.70-TL, symbol easyeda2kicad:LM2596SX-5.0_NOPB
- renumbered C900 to C11, C901 to C12, C903 to C14, L20 to L2, R80 to R10, R81 to R9, RV20 to RV1
Connections:
- net LM2596_VIN: now also J6.1 (Pin_1), U6.1 (VIN)
- net LM2596_VOUT: no longer C14.1, L2.2, R10.1, RV1.1
- net SW: now also D5.1 (K), U6.2 (OUT)
- net at R9.1, RV1.2, RV1.3: now also U6.4 (FB)
- net at R10.2: now also D6.2 (A)
- net GND renamed LM2596_GND
- net LM2596_GND: now also C13.2, D5.2 (A), D6.1 (K), J7.1 (Pin_1), J9.1 (Pin_1), U6.3 (GND), U6.5 (~{ON}/OFF), U6.6 (GND)
- new net: C13.1, C14.1, J8.1 (Pin_1), L2.2, R10.1, RV1.1
Other:
- moved on the sheet: C11, C12, C14, L2, R10, R9, RV1
