File: Final/final.kicad_sch (KiCad schematic)
At the start: 232 parts, among them J1 2.54-1*6PHeader-RA, J10 Conn_01x02, J11 Conn_01x04, J2 USB_C_Receptacle_PowerOnly_6P, P1 Header-Male-2.54_2x2, P10 1.27mm/1*3p, P11 1.27mm/1*3p, P2 Header-Male-2.54_2x2, P3 1.27mm/1*3p, P4 1.27mm/1*3p, P5 1.27mm/1*3p, P6 1.27mm/1*3p, P7 1.27mm/1*3p, P8 1.27mm/1*3p, P9 1.27mm/1*3p, Q1 2N7002, Q10 AO3400A, Q11 AO3401A, Q2 CJQ4435, Q3 currentmirror, Q4 BSS84, Q5 AO4892, Q6 AO3401A, Q7 AO3401A, Q8 CJQ4435, Q9 AO3400A, SW1 TS-1088R-02026, U1 MAX17048G+T10, U10 BQ25606RGER, U11 Battery Input, U12 BQ24170RGYR, U13 TPS54302DDCR_C311983, U14 NTC10K/0805/F, U15 BQ76920PW, U16 NTC10K/0805/F, U17 HUSB238_002DD, U19 TPS54302DDCR_C311983, U2 MT3608, U20 TPS54302DDCR_C311983, U21 MCP73871, U22 SRP4020TA-1R0M, U3 MT3608, U4 TPL5110DDCT, U5 BQ25606RGER, U6 MT3608, U7 Z-21320110021001, U8 MAX3232CDBR, U9 ADS1115IDGSR

Commit message: added a final PCB folder
Co-authored-by: Copilot <copilot@github.com>
Parts:
- removed C29, C37, C43: 10uF, PCM_JLCPCB:C_0603, symbol PCM_JLCPCB-Capacitors:0603,10uF
- removed C32, C33, C34, C38, C44, C45: 100nF, PCM_JLCPCB:C_0603, symbol PCM_JLCPCB-Capacitors:0603,100nF
- removed C35, C36, C40, C41, C46, C47: 22uF, PCM_JLCPCB:C_0603, symbol PCM_JLCPCB-Capacitors:0603,22uF
- removed C39: 47pF, PCM_JLCPCB:C_0603, symbol PCM_JLCPCB-Capacitors:0603,47pF
- removed C48: 75pf, easyeda2kicad:C0603, symbol easyeda2kicad:0603CG750J500NT
- removed C49: 100pF, PCM_JLCPCB:C_0603, symbol PCM_JLCPCB-Capacitors:0603,100pF
- removed L5: 10uh, easyeda2kicad:IND-SMD_L7.5-W6.6, symbol easyeda2kicad:CKST0605-10UH_M
- removed L6: 6.8uh, easyeda2kicad:IND-SMD_L12.3-W12.3_SMDRI127, symbol easyeda2kicad:SMDRI127-6R8NT
- removed L7: 15uh, easyeda2kicad:IND-SMD_L10.4-W10.3, symbol easyeda2kicad:SMDRH104R-150MT
- removed P4, P8, P9: 1.27mm/1*3p, easyeda2kicad:HDR-TH_3P-P1.27-V-M-1, symbol easyeda2kicad:1.27mm_1*3p
- removed R37, R44, R49: 49.9kΩ, PCM_JLCPCB:R_0603, symbol PCM_JLCPCB-Resistors:0603,49.9kΩ
- removed R38, R45, R50: 100kΩ, PCM_JLCPCB:R_0603, symbol PCM_JLCPCB-Resistors:0603,100kΩ
- removed R40, R42, R47: 511k, easyeda2kicad:R0805, symbol easyeda2kicad:0805W8F5113T5E
- removed R41, R43, R48: 105k, easyeda2kicad:R0603, symbol easyeda2kicad:0603WAF1053T5E
- removed R46: 3kΩ, PCM_JLCPCB:R_0603, symbol PCM_JLCPCB-Resistors:0603,3kΩ
- removed R51: 13.3k, easyeda2kicad:R0805, symbol easyeda2kicad:0805W8F1332T5E
- removed R52: 22kΩ, PCM_JLCPCB:R_0603, symbol PCM_JLCPCB-Resistors:0603,22kΩ
- removed R53: 2.2kΩ, PCM_JLCPCB:R_0603, symbol PCM_JLCPCB-Resistors:0603,2.2kΩ
- removed U13, U19, U20: TPS54302DDCR_C311983, easyeda2kicad:SOT-23-6_L2.9-W1.6-P0.95-LS2.8-BL, symbol easyeda2kicad:TPS54302DDCR_C311983
Other:
- note removed: "For BUCK: Vout = Vref*(R2/R3+1)"
- note removed: "Vout = 0.596*(100/13.3+1)"
- note removed: "Vout = 0.596*(100/22+1)"
- note removed: "Vout = 0.596*(100/5.2+1)"
