File: TESTPCB/charging-circuit/sheets/_backup_before_netlabel_conversion/06_v1_ic.kicad_sch (KiCad schematic)
At the start: 16 parts, among them P10 1.27mm/1*3p, U21 MCP73871

Commit message: Fixed formatting issues, now the hierachal sheets are all labeled as net labels and when we want to expose their pins we will make them into hierchal or global pins
Changed lines of the file:
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@@
 		)
 	)
-	(label "V1GND"
+	(global_label "V1GND"
+		(shape bidirectional)
 		(at 93.98 109.22 270)
 		(effects
@@
 			(justify right bottom)
 		)
-	)
-	(label "V1VBUS"
+		(property "Intersheetrefs" "${INTERSHEET_REFS}"
+			(at 93.98 109.22 0)
+			(effects
+				(font
+					(size 1.27 1.27)
+				)
+				(hide yes)
+			)
+		)
+	)
+	(global_label "V1VBUS"
+		(shape bidirectional)
 		(at 93.98 55.88 90)
 		(effects
@@
 			(justify left bottom)
 		)
-	)
-	(label "V1GND"
+		(property "Intersheetrefs" "${INTERSHEET_REFS}"
+			(at 93.98 55.88 0)
+			(effects
+				(font
+					(size 1.27 1.27)
+				)
+				(hide yes)
+			)
+		)
+	)
+	(global_label "V1GND"
+		(shape bidirectional)
 		(at 44.45 76.2 270)
 		(effects
@@
 			(justify right bottom)
 		)
-	)
-	(label "V1GND"
+		(property "Intersheetrefs" "${INTERSHEET_REFS}"
+			(at 44.45 76.2 0)
+			(effects
+				(font
+					(size 1.27 1.27)
+				)
+				(hide yes)
+			)
+		)
+	)
+	(global_label "V1GND"
+		(shape bidirectional)
 		(at 81.28 57.15 270)
 		(effects
@@
 			(justify right bottom)
 		)
-	)
-	(label "V1GND"
+		(property "Intersheetrefs" "${INTERSHEET_REFS}"
+			(at 81.28 57.15 0)
+			(effects
+				(font
+					(size 1.27 1.27)
+				)
+				(hide yes)
+			)
+		)
+	)
+	(global_label "V1GND"
+		(shape bidirectional)
 		(at 76.2 76.2 180)
 		(effects
@@
 			(justify right bottom)
 		)
-	)
-	(label "V1VSYS"
+		(property "Intersheetrefs" "${INTERSHEET_REFS}"
+			(at 76.2 76.2 0)
+			(effects
+				(font
+					(size 1.27 1.27)
+				)
+				(hide yes)
+			)
+		)
+	)
+	(global_label "V1VSYS"
+		(shape bidirectional)
 		(at 125.73 52.07 0)
 		(effects
@@
 			(justify left bottom)
 		)
-	)
-	(label "V1GND"
+		(property "Intersheetrefs" "${INTERSHEET_REFS}"
+			(at 125.73 52.07 0)
+			(effects
+				(font
+					(size 1.27 1.27)
+				)
+				(hide yes)
+			)
+		)
+	)
+	(global_label "V1GND"
+		(shape bidirectional)
 		(at 66.04 60.96 0)
 		(effects
@@
 			(justify left bottom)
 		)
-	)
-	(label "V1GND"
+		(property "Intersheetrefs" "${INTERSHEET_REFS}"
+			(at 66.04 60.96 0)
+			(effects
+				(font
+					(size 1.27 1.27)
+				)
+				(hide yes)
+			)
+		)
+	)
+	(global_label "V1GND"
+		(shape bidirectional)
 		(at 128.27 76.2 270)
 		(effects
@@
 			(justify right bottom)
 		)
-	)
-	(label "V1VBUS"
+		(property "Intersheetrefs" "${INTERSHEET_REFS}"
+			(at 128.27 76.2 0)
+			(effects
+				(font
+					(size 1.27 1.27)
+				)
+				(hide yes)
+			)
+		)
+	)
+	(global_label "V1VBUS"
+		(shape bidirectional)
 		(at 76.2 83.82 180)
 		(effects
@@
 			(justify right bottom)
 		)
-	)
-	(label "V1VBUS"
+		(property "Intersheetrefs" "${INTERSHEET_REFS}"
+			(at 76.2 83.82 0)
+			(effects
+				(font
+					(size 1.27 1.27)
+				)
+				(hide yes)
+			)
+		)
+	)
+	(global_label "V1VBUS"
+		(shape bidirectional)
 		(at 66.04 55.88 0)
 		(effects
@@
 			(justify left bottom)
 		)
-	)
-	(label "V1GND"
+		(property "Intersheetrefs" "${INTERSHEET_REFS}"
+			(at 66.04 55.88 0)
+			(effects
+				(font
+					(size 1.27 1.27)
+				)
+				(hide yes)
+			)
+		)
+	)
+	(global_label "V1GND"
+		(shape bidirectional)
 		(at 49.53 86.36 180)
 		(effects
@@
 			(justify right bottom)
 		)
-	)
-	(label "V1GND"
+		(property "Intersheetrefs" "${INTERSHEET_REFS}"
+			(at 49.53 86.36 0)
+			(effects
+				(font
+					(size 1.27 1.27)
+				)
+				(hide yes)
+			)
+		)
+	)
+	(global_label "V1GND"
+		(shape bidirectional)
 		(at 115.57 59.69 270)
 		(effects
@@
 			(justify right bottom)
 		)
-	)
-	(label "V1VSYS"
+		(property "Intersheetrefs" "${INTERSHEET_REFS}"
+			(at 115.57 59.69 0)
+			(effects
+				(font
+					(size 1.27 1.27)
+				)
+				(hide yes)
+			)
+		)
+	)
+	(global_label "V1VSYS"
+		(shape bidirectional)
 		(at 66.04 58.42 0)
 		(effects
@@
 			(justify left bottom)
 		)
-	)
-	(label "V1VBUS"
+		(property "Intersheetrefs" "${INTERSHEET_REFS}"
+			(at 66.04 58.42 0)
+			(effects
+				(font
+					(size 1.27 1.27)
+				)
+				(hide yes)
+			)
+		)
+	)
+	(global_label "V1VBUS"
+		(shape bidirectional)
 		(at 72.39 101.6 180)
 		(effects
@@
 			(justify right bottom)
 		)
-	)
-	(label "V1VSYS"
+		(property "Intersheetrefs" "${INTERSHEET_REFS}"
+			(at 72.39 101.6 0)
+			(effects
+				(font
+					(size 1.27 1.27)
+				)
+				(hide yes)
+			)
+		)
+	)
+	(global_label "V1VSYS"
+		(shape bidirectional)
 		(at 142.24 96.52 0)
 		(effects
@@
 			(justify left bottom)
 		)
-	)
-	(label "V1VBAT"
+		(property "Intersheetrefs" "${INTERSHEET_REFS}"
+			(at 142.24 96.52 0)
+			(effects
+				(font
+					(size 1.27 1.27)
+				)
+				(hide yes)
+			)
+		)
+	)
+	(global_label "V1VBAT"
+		(shape bidirectional)
 		(at 144.78 67.31 0)
 		(effects
@@
 			(justify left bottom)
 		)
-	)
-	(label "V1VBUS"
+		(property "Intersheetrefs" "${INTERSHEET_REFS}"
+			(at 144.78 67.31 0)
+			(effects
+				(font
+					(size 1.27 1.27)
+				)
+				(hide yes)
+			)
+		)
+	)
+	(global_label "V1VBUS"
+		(shape bidirectional)
 		(at 44.45 60.96 180)
 		(effects
@@
 			(justify right bottom)
 		)
-	)
+		(property "Intersheetrefs" "${INTERSHEET_REFS}"
+			(at 44.45 60.96 0)
+			(effects
+				(font
+					(size 1.27 1.27)
+				)
+				(hide yes)
+			)
+		)
+	)
