File: TESTPCB/charging-circuit/sheets/_backup_before_netlabel_conversion/18_lm2596_5V_buck.kicad_sch (KiCad schematic)
At the start: 13 parts, among them J3 Conn_01x01_Pin, J4 Conn_01x01_Pin, J5 Conn_01x01_Pin, J6 Conn_01x01_Pin, U18 LM2596SX-5.0/NOPB

Commit message: Fixed formatting issues, now the hierachal sheets are all labeled as net labels and when we want to expose their pins we will make them into hierchal or global pins
Changed lines of the file:
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@@
-		)
-	)
-	(label "LM2596_5V_VOUT"
-		(at 207.01 93.98 0)
-		(effects
-			(font
-				(size 1.27 1.27)
-			)
-			(justify left bottom)
 		)
 	)
@@
 		)
 	)
-	(label "LM2596_5V_VIN"
+	(global_label "LM2596_5V_VOUT"
+		(shape bidirectional)
+		(at 207.01 93.98 0)
+		(effects
+			(font
+				(size 1.27 1.27)
+			)
+			(justify left bottom)
+		)
+		(property "Intersheetrefs" "${INTERSHEET_REFS}"
+			(at 207.01 93.98 0)
+			(effects
+				(font
+					(size 1.27 1.27)
+				)
+				(hide yes)
+			)
+		)
+	)
+	(global_label "LM2596_5V_VIN"
+		(shape bidirectional)
 		(at 81.28 88.9 0)
 		(effects
@@
 			(justify left bottom)
 		)
+		(property "Intersheetrefs" "${INTERSHEET_REFS}"
+			(at 81.28 88.9 0)
+			(effects
+				(font
+					(size 1.27 1.27)
+				)
+				(hide yes)
+			)
+		)
 	)
