File: TESTPCB/charging-circuit/sheets/04_sleepmosfet.kicad_sch (KiCad schematic)
At the start: 8 parts, among them P3 1.27mm/1*3p, Q8 CJQ4435, U4 TPL5110DDCT

Commit message: sunday
Parts:
- removed C3: 100nF, PCM_JLCPCB:C_0603, symbol PCM_JLCPCB-Capacitors:0603,100nF
- removed P3: 1.27mm/1*3p, easyeda2kicad:HDR-TH_3P-P1.27-V-M-1, symbol easyeda2kicad:1.27mm_1*3p
- removed Q8: CJQ4435, easyeda2kicad:SOP-8_L5.0-W4.0-P1.27-LS6.2-BL, symbol easyeda2kicad:CJQ4435
- removed R54: RM065-204(200K), easyeda2kicad:RES-ADJ-TH_3P-L7.3-W6.4-P5.00-R, symbol easyeda2kicad:RM065-204(200K)
- removed R8, R9: 10kΩ, PCM_JLCPCB:R_0603, symbol PCM_JLCPCB-Resistors:0603,10kΩ
- removed RPROG1: 1kΩ, PCM_JLCPCB:R_0603, symbol PCM_JLCPCB-Resistors:0603,1kΩ
- removed U4: TPL5110DDCT, easyeda2kicad:TSOT-23-6_L2.9-W1.6-P0.95-LS2.8-BR, symbol easyeda2kicad:TPL5110DDCT
- added C65: 100nF, PCM_JLCPCB:C_0603, symbol PCM_JLCPCB-Capacitors:0603,100nF
- added Q12, Q18, Q19, Q8: 2N7002, easyeda2kicad:SOT-23-3_L2.9-W1.3-P1.90-LS2.4-BR, symbol easyeda2kicad:2N7002
- added Q13, Q14, Q20: CJQ4435, easyeda2kicad:SOP-8_L5.0-W4.0-P1.27-LS6.2-BL, symbol easyeda2kicad:CJQ4435
- added R17, R22, R23, R28, R29: 10kΩ, PCM_JLCPCB:R_0603, symbol PCM_JLCPCB-Resistors:0603,10kΩ
- added R24, R25, R27: 100kΩ, PCM_JLCPCB:R_0603, symbol PCM_JLCPCB-Resistors:0603,100kΩ
- added R68: RM065-204(200K), easyeda2kicad:RES-ADJ-TH_3P-L7.3-W6.4-P5.00-R, symbol easyeda2kicad:RM065-204(200K)
- added RPROG6, RPROG7: 1kΩ, PCM_JLCPCB:R_0603, symbol PCM_JLCPCB-Resistors:0603,1kΩ
- added U19: TPL5110DDCT, easyeda2kicad:TSOT-23-6_L2.9-W1.6-P0.95-LS2.8-BR, symbol easyeda2kicad:TPL5110DDCT
Connections:
- new net: Q12.3 (D), Q13.4 (G), R22.1
- new net: Q18.3 (D), Q19.1 (G), R24.2
- new net: Q14.4 (G), Q8.3 (D), R17.1
- new net: Q19.3 (D), Q20.4 (G), R25.1
- new net: R68.1, U19.3 (DELAY/M_DRV)
- new net 12VOUT: Q20.5 (D), Q20.6 (D), Q20.7 (D), Q20.8 (D), R27.2
- new net 5EN: Q14.5 (D), Q14.6 (D), Q14.7 (D), Q14.8 (D), RPROG6.1
- new net SLP12V: Q14.1 (S), Q14.2 (S), Q14.3 (S), Q20.1 (S), Q20.2 (S), Q20.3 (S), R17.2, R25.2
- new net SLP3V3: Q13.1 (S), Q13.2 (S), Q13.3 (S), R22.2, R24.1, U19.1 (VDD), U19.6 (EN/ONE_SHOT)
- new net SLPDRV: Q18.1 (G), Q8.1 (G), R29.1, U19.5 (DRV)
- new net SLPGND: C65.2, Q12.2 (S), Q18.2 (S), Q19.2 (S), Q8.2 (S), R23.2, R27.1, R28.1, R29.2, RPROG6.2, RPROG7.2, U19.2 (GND)
- new net SLPRASPI: Q12.1 (G), R28.2
- new net SLPSIG: C65.1, Q13.5 (D), Q13.6 (D), Q13.7 (D), Q13.8 (D), R23.1, RPROG7.1, U19.4 (DONE)
Other:
- note added: "n, pmos driver for enable pin of lmk2596 5 volts"
- note added: "n, pmos driver for raspi to tpl5110 side (3.3 Volts NOT 12)"
- note added: "n,n,pmos driver for 12Volts (directly from battery)"
- note removed: "potentiometer, leave floating"
