File: TESTPCB/charging-circuit/sheets/05_fuelgauge.kicad_sch (KiCad schematic)
At the start: 2 parts, among them P2 Header-Male-2.54_2x2, U1 MAX17048G+T10

Commit message: sunday
Connections:
- net FUELBAT: no longer U1.3 (VDD)
- new net FUEL3V3: U1.3 (VDD)
