File: TESTPCB/charging-circuit/sheets/18_lm2596_adj_buck.kicad_sch (KiCad schematic)
At the start: 15 parts, among them J20 Conn_01x01_Pin, J21 Conn_01x01_Pin, J22 Conn_01x01_Pin, J23 Conn_01x01_Pin, U30 LM2596S-ADJ

Commit message: Fixed formatting issues, now the hierachal sheets are all labeled as net labels and when we want to expose their pins we will make them into hierchal or global pins
Changed lines of the file:
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@@
+		)
+	)
+	(label "LM2596_VOUT"
+		(at 219.71 93.98 0)
+		(effects
+			(font
+				(size 1.27 1.27)
+			)
+			(justify left bottom)
 		)
 	)
@@
 		)
 	)
-	(global_label "LM2596_VOUT"
-		(shape bidirectional)
-		(at 219.71 93.98 0)
-		(effects
-			(font
-				(size 1.27 1.27)
-			)
-			(justify left bottom)
-		)
-		(property "Intersheetrefs" "${INTERSHEET_REFS}"
-			(at 219.71 93.98 0)
-			(effects
-				(font
-					(size 1.27 1.27)
-				)
-				(hide yes)
-			)
-		)
-	)
-	(global_label "LM2596_VIN"
-		(shape bidirectional)
+	(label "LM2596_VIN"
 		(at 81.28 88.9 0)
 		(effects
@@
 			(justify left bottom)
 		)
-		(property "Intersheetrefs" "${INTERSHEET_REFS}"
-			(at 81.28 88.9 0)
-			(effects
-				(font
-					(size 1.27 1.27)
-				)
-				(hide yes)
-			)
-		)
 	)
