File: V4/charging-circuit/sheets/18_lm2596_5V_buck.kicad_sch (KiCad schematic)
At the start: 10 parts, among them U21 LM2596SX-5.0/NOPB

Commit message: schem
Parts:
- removed R6: 4.7k, easyeda2kicad:R0805, symbol easyeda2kicad:0805W8F4701T5E
- removed U21: LM2596SX-5.0/NOPB, easyeda2kicad:TO-263-5_L10.2-W8.9-P1.70-TL, symbol easyeda2kicad:LM2596SX-5.0_NOPB
- added R2: 4.7kΩ, PCM_JLCPCB:R_0805, symbol PCM_JLCPCB-Resistors:0805,4.7kΩ
- added U6: LM2596SX-5.0/NOPB, easyeda2kicad:TO-263-5_L10.2-W8.9-P1.70-TL, symbol easyeda2kicad:LM2596SX-5.0_NOPB
Connections:
- net 5EN: now also U6.5 (~{ON}/OFF)
- net 5VIN+: now also U6.1 (VIN)
- net 5VIN-: now also U6.3 (GND), U6.6 (GND)
- net 5VOUT+: now also R2.1, U6.4 (FB)
- net SW: now also U6.2 (OUTPUT)
- net at D10.2: now also R2.2
