File: V4/charging-circuit/sheets/14_3s_ic.kicad_sch (KiCad schematic)
At the start: 24 parts, among them U1 IP2326, U3 90KR

Commit message: schem
Parts:
- removed R2, R3: 0805W8F5102T5E, easyeda2kicad:R0805, symbol easyeda2kicad:0805W8F5102T5E
- removed U3: 90KR, easyeda2kicad:R0805, symbol easyeda2kicad:HOAR0805-1_8W-90KR-0.25%-TCR50
- added R12: 62kΩ, PCM_JLCPCB:R_0805, symbol PCM_JLCPCB-Resistors:0805,62kΩ
- added R18, R19: 51kΩ, PCM_JLCPCB:R_0805, symbol PCM_JLCPCB-Resistors:0805,51kΩ
Connections:
- net BAT-: now also R12.1, R18.1
- net ICEN: now also R19.2
- net ICVBUS: now also R19.1
- net at U1.11 (ISET): now also R12.2
- net at U1.4 (NTC): now also R18.2

Commit message: finished
Changed lines of the file:
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@@
+		)
+	)
+	(hierarchical_label "GND"
+		(shape input)
+		(at 153.67 125.73 0)
+		(effects
+			(font
+				(size 1.27 1.27)
+			)
+			(justify left)
 		)
 	)
