File: V4/charging-circuit/sheets/17_dsub_rs232.kicad_sch (KiCad schematic)
At the start: 8 parts, among them U10 MAX3232CDBR

Commit message: schem
Parts:
- removed DSub1: DR-15P圆针公蓝色, easyeda2kicad:D-SUB-TH_BOOMELE_DR-15P, symbol easyeda2kicad:DR-15P圆针公蓝色
Other:
- moved on the sheet: DSub2

Commit message: tuesday
Parts:
- added TP14, TP22: VBUS, Connector_PinHeader_2.54mm:PinHeader_1x01_P2.54mm_Vertical, symbol Connector:TestPoint
Connections:
- net UART_RX_13V is gone; now on net RX: DSub2.1, U10.13 (RIN1)
- net UART_TX_13V is gone; now on net TX: DSub2.2, U10.14 (DOUT1)
Changed lines of the file:
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@@
 		)
 	)
-	(label "TX"
+	(label "UART_TX_13V"
 		(at 52.07 68.58 0)
 		(effects
@@
 		)
 	)
-	(label "RX"
+	(label "UART_RX_13V"
 		(at 52.07 71.12 0)
 		(effects
@@
 		)
 	)
+	(symbol
+		(lib_id "Connector:TestPoint")
+		(at 0.762 5.5937 0)
+		(unit 1)
+		(body_style 1)
+		(exclude_from_sim no)
+		(in_bom yes)
+		(on_board yes)
+		(in_pos_files yes)
+		(dnp no)
+		(fields_autoplaced yes)
+		(property "Reference" "TP14"
+			(at 3.302 1.0216 0)
+			(show_name no)
+			(do_not_autoplace no)
+			(effects
+				(font
+					(size 1.27 1.27)
+				)
+				(justify left)
+			)
+		)
+		(property "Value" "VBUS"
+			(at 3.302 3.5616 0)
+			(show_name no)
+			(do_not_autoplace no)
+			(effects
+				(font
+					(size 1.27 1.27)
+				)
+				(justify left)
+			)
+		)
+		(property "Footprint" "Connector_PinHeader_2.54mm:PinHeader_1x01_P2.54mm_Vertical"
+			(at 5.842 5.5937 0)
+			(hide yes)
+			(show_name no)
+			(do_not_autoplace no)
+			(effects
+				(font
+					(size 1.27 1.27)
+				)
+			)
+		)
+		(property "Datasheet" ""
+			(at 5.842 5.5937 0)
+			(hide yes)
+			(show_name no)
+			(do_not_autoplace no)
+			(effects
+				(font
+					(size 1.27 1.27)
+				)
+			)
+		)
+		(property "Description" "test point"
+			(at 0.762 5.5937 0)
+			(hide yes)
+			(show_name no)
+			(do_not_autoplace no)
+			(effects
+				(font
+					(size 1.27 1.27)
+				)
+			)
+		)
+		(pin "1"
+		)
+		(instances
+			(project "charging-circuit"
+				(path "/529bc8a5-ffae-43ac-972d-caccc3afab85/b2555034-0671-4d54-9747-cad620ff9682"
+					(reference "TP14")
+					(unit 1)
+				)
+			)
+		)
+	)
+	(symbol
+		(lib_id "Connector:TestPoint")
+		(at 7.112 11.9437 0)
+		(unit 1)
+		(body_style 1)
+		(exclude_from_sim no)
+		(in_bom yes)
+		(on_board yes)
+		(in_pos_files yes)
+		(dnp no)
+		(fields_autoplaced yes)
+		(property "Reference" "TP22"
+			(at 9.652 7.3716 0)
+			(show_name no)
+			(do_not_autoplace no)
+			(effects
+				(font
+					(size 1.27 1.27)
+				)
+				(justify left)
+			)
+		)
+		(property "Value" "VBUS"
+			(at 9.652 9.9116 0)
+			(show_name no)
+			(do_not_autoplace no)
+			(effects
+				(font
+					(size 1.27 1.27)
+				)
+				(justify left)
+			)
+		)
+		(property "Footprint" "Connector_PinHeader_2.54mm:PinHeader_1x01_P2.54mm_Vertical"
+			(at 12.192 11.9437 0)
+			(hide yes)
+			(show_name no)
+			(do_not_autoplace no)
+			(effects
+				(font
+					(size 1.27 1.27)
+				)
+			)
+		)
+		(property "Datasheet" ""
+			(at 12.192 11.9437 0)
+			(hide yes)
+			(show_name no)
+			(do_not_autoplace no)
+			(effects
+				(font
+					(size 1.27 1.27)
+				)
+			)
+		)
+		(property "Description" "test point"
+			(at 7.112 11.9437 0)
+			(hide yes)
+			(show_name no)
+			(do_not_autoplace no)
+			(effects
+				(font
+					(size 1.27 1.27)
+				)
+			)
+		)
+		(pin "1"
+		)
+		(instances
+			(project "charging-circuit"
+				(path "/529bc8a5-ffae-43ac-972d-caccc3afab85/b2555034-0671-4d54-9747-cad620ff9682"
+					(reference "TP22")
+					(unit 1)
+				)
+			)
+		)
+	)
