File: V4/charging-circuit/charging-circuit.kicad_pcb (KiCad board)
At the start: 2 copper layers, 82.6 x 94.6 mm, 270 parts, among them J1 2.54-1*6PHeader-RA, J10 Conn_01x02, J11 Conn_01x04, J2 USB_C_Receptacle_PowerOnly_6P, P1 Header-Male-2.54_2x2, P10 1.27mm/1*3p, P11 1.27mm/1*3p, P2 Header-Male-2.54_2x2, P3 1.27mm/1*3p, P4 1.27mm/1*3p, P5 1.27mm/1*3p, P6 1.27mm/1*3p, P7 1.27mm/1*3p, P8 1.27mm/1*3p, P9 1.27mm/1*3p, Q1 2N7002, Q10 AO3400A, Q11 AO3401A, Q2 CJQ4435, Q3 currentmirror, Q4 BSS84, Q5 AO4892, Q6 AO3401A, Q7 AO3401A, Q8 CJQ4435, Q9 AO3400A, SW1 TS-1088R-02026, U1 MAX17048G+T10, U10 BQ25606RGER, U11 Battery Input, U12 BQ24170RGYR, U13 TPS54302DDCR_C311983, U14 NTC10K/0805/F, U15 BQ76920PW, U16 NTC10K/0805/F, U17 HUSB238_002DD, U19 TPS54302DDCR_C311983, U2 MT3608, U20 TPS54302DDCR_C311983, U21 MCP73871, U22 SRP4020TA-1R0M, U3 MT3608, U4 TPL5110DDCT, U5 BQ25606RGER, U6 MT3608, U7 Z-21320110021001, U8 MAX3232CDBR, U9 ADS1115IDGSR

Commit message: schem
Parts:
- removed the ? at (54.3, 64.3)
- removed the ? at (41.3, 64.3)
- removed the ? at (93.5, 85.7)
- removed the ? at (67.5, 85.7)
- removed the ? at (104.8, 64.3)
- removed the ? at (67.5, 43.5)
- removed the ? at (57.7, 53.9)
- removed the ? at (60.1, 92.6)
- removed the ? at (76.2, 92.6)
- removed the ? at (94.0, 53.9)
- removed the ? at (72.0, 74.8)
- removed the ? at (105.0, 85.7)
- removed the ? at (58.5, 31.5)
- removed the ? at (80.5, 43.5)
- removed the ? at (87.0, 31.4)
- removed the ? at (93.3, 64.3)
- removed the ? at (43.0, 106.7)
- removed the ? at (54.5, 85.7)
- removed the ? at (94.5, 93.0)
- removed the ? at (41.5, 85.7)
- removed the ? at (44.1, 31.6)
- removed the ? at (80.5, 85.7)
- removed the ? at (72.7, 31.4)
- removed the ? at (93.5, 43.5)
- removed the ? at (44.5, 74.8)
- removed the ? at (43.0, 92.7)
- removed the ? at (67.3, 64.3)
- removed the ? at (94.5, 107.0)
- removed the ? at (105.0, 43.5)
- removed the ? at (30.8, 64.3)
- removed the ? at (60.1, 106.6)
- removed the ? at (64.5, 74.8)
- removed the ? at (41.5, 43.5)
- removed the ? at (76.2, 106.6)
- removed the ? at (31.0, 85.7)
- removed the ? at (80.3, 64.3)
- removed the ? at (54.5, 43.5)
- removed C1: 22uf, easyeda2kicad:C0805
- removed C17, C20, C32, C34, C44, C45, C54, C57, C61, C_sense1, C_sense2, C_sense3: 100nF, PCM_JLCPCB:C_0603
- removed C26, C28: 1uF, PCM_JLCPCB:C_0402
- removed C30: 1uF, PCM_JLCPCB:C_1206
- removed C31, C42, C53, C55, C70, C71, C9, Cc0, Cc1: 1uF, PCM_JLCPCB:C_0603
- removed C37, C43, C50: 10uF, PCM_JLCPCB:C_0603
- removed C41, C46, C47: 22uF, PCM_JLCPCB:C_0603
- removed C48: 75pf, easyeda2kicad:C0603
- removed C49: 100pF, PCM_JLCPCB:C_0603
- removed C51, C52: 4.7uF, PCM_JLCPCB:C_0603
- removed C56: 47nF, PCM_JLCPCB:C_0603
- removed C58, C72: 10uF, PCM_JLCPCB:C_1206
- removed C59: 22uF, PCM_JLCPCB:C_0805
- removed Cin1: 2.2uF, PCM_JLCPCB:C_0805
- removed D100: MBR0530, easyeda2kicad:SOD-123_L2.8-W1.8-LS3.7-RD
- removed D19: B0530W, PCM_JLCPCB:D_SOD-123
- removed D4: SS34, PCM_JLCPCB:D_SMA
- removed H11, H2: 77311-462K05LF, easyeda2kicad:HDR-TH_5P-P2.54-V-M
- removed H3, H4, H9: Header-Male-2.54_1x6, easyeda2kicad:HDR-TH_6P-P2.54-V-M-1
- removed H5, H6, H7, H8: 68000-102HLF, easyeda2kicad:HDR-TH_2P-P2.54-V-M-1
- removed J1: 2.54-1*6PHeader-RA, easyeda2kicad:HDR-TH_6P-P2.54-H-M-W10.0
- removed J10: Conn_01x02, Connector_PinHeader_2.54mm:PinHeader_1x02_P2.54mm_Vertical
- removed J11: Conn_01x04, Connector_PinHeader_2.54mm:PinHeader_1x04_P2.54mm_Vertical
- removed J2: USB_C_Receptacle_PowerOnly_6P, easyeda2kicad:TYPE-C-SMD_TYPE-C-6P
- removed L2: 22uH, easyeda2kicad:IND-SMD_L7.5-W7.5
- removed L6: 6.8uh, easyeda2kicad:IND-SMD_L12.3-W12.3_SMDRI127
- removed L7: 15uh, easyeda2kicad:IND-SMD_L10.4-W10.3
- removed L8: 2.2uH, easyeda2kicad:IND-SMD_L6.7-W6.6
- removed P1: Header-Male-2.54_2x2, easyeda2kicad:HDR-TH_4P-P2.54-V-M-R2-C2-S2.54-1
- removed P11, P6, P7, P8, P9: 1.27mm/1*3p, easyeda2kicad:HDR-TH_3P-P1.27-V-M-1
- removed Q1: 2N7002, easyeda2kicad:SOT-23-3_L2.9-W1.3-P1.90-LS2.4-BR
- removed Q10, Q9: AO3400A, PCM_JLCPCB:Q_SOT-23
- removed Q2, Q8: CJQ4435, easyeda2kicad:SOP-8_L5.0-W4.0-P1.27-LS6.2-BL
- removed Q3: currentmirror, easyeda2kicad:SOT-363-6_L2.2-W1.3-P0.65-LS2.1-BL
- removed Q4: BSS84, Package_TO_SOT_SMD:SOT-23
- removed Q6, Q7: AO3401A, easyeda2kicad:SOT-23_L2.9-W1.3-P1.90-LS2.4-BR
- removed R12, R13, R30, R35: 5.1kΩ, PCM_JLCPCB:R_0603
- removed R17, R20: 2.2kΩ, PCM_JLCPCB:R_0603
- removed R18: 6.8kΩ, PCM_JLCPCB:R_0603
- removed R19: 2kΩ, PCM_JLCPCB:R_0603
- removed R27: 5.23kohm, easyeda2kicad:R0603
- removed R28: 30.1kohm, easyeda2kicad:R0603
- removed R29, RPROG3: 10kΩ, PCM_JLCPCB:R_0603
- removed R34: 330kΩ, PCM_JLCPCB:R_0603
- removed R36: 12kΩ, PCM_JLCPCB:R_0603
- removed R42: 511k, easyeda2kicad:R0805
- removed R55: 3296W-1-504LF, easyeda2kicad:RES-ADJ-TH_3296W
- removed R56, R57, R58: 470Ω, PCM_JLCPCB:R_0603
- removed R59: 110kΩ, PCM_JLCPCB:R_0603
- removed R60: 1MΩ, PCM_JLCPCB:R_0603
- removed R61, R76: 100kΩ, PCM_JLCPCB:R_0603
- removed R62: 30.1k, easyeda2kicad:R0603
- removed R63, R75: 4.02k, easyeda2kicad:R0603
- removed R64: 1.5kΩ, PCM_JLCPCB:R_0402
- removed R65, RPROG1, RPROG2, RPROG5: 1kΩ, PCM_JLCPCB:R_0603
- removed R66: 33kΩ, PCM_JLCPCB:R_0402
- removed R7: 32.4k, easyeda2kicad:R0603
- removed R77: 49.9kΩ, PCM_JLCPCB:R_0603
- removed R_AC1, R_AC2: 10m, easyeda2kicad:R1206
- removed R_sense1, R_sense2, Rc0, Rc1, Rc2, Rc3: 100Ω, PCM_JLCPCB:R_0603
- removed Rin1: 2Ω, PCM_JLCPCB:R_0603
- removed Rsense1: LTR18EZPFSR015, easyeda2kicad:R0612
- removed SW1: TS-1088R-02026, easyeda2kicad:SW-SMD_L3.9-W3.0-P4.45
- removed U11: Battery Input, easyeda2kicad:CONN-TH_S2B-PH-K-S-GW
- removed U13, U20: TPS54302DDCR_C311983, easyeda2kicad:SOT-23-6_L2.9-W1.6-P0.95-LS2.8-BL
- removed U14, U16: NTC10K/0805/F, easyeda2kicad:R0805
- removed U15: BQ76920PW, Package_SO:TSSOP-20_4.4x6.5mm_P0.65mm
- removed U17: HUSB238_002DD, easyeda2kicad:DFN-10_L3.0-W3.0-P0.50-BL-EP2.5
- removed U21: MCP73871, easyeda2kicad:QFN-20_L4.0-W4.0-P0.5-BL-EP
- removed U22: SRP4020TA-1R0M, easyeda2kicad:IND-SMD_L4.5-W4.1_SRP4020TA
- removed U5: BQ25606RGER, easyeda2kicad:VQFN-24_L4.0-W4.0-P0.50-TL-EP2.8
- removed U8: MAX3232CDBR, easyeda2kicad:SSOP-16_L6.2-W5.3-P0.65-LS7.8-BL
- removed U9: ADS1115IDGSR, easyeda2kicad:MSOP-10_L3.0-W3.0-P0.50-LS5.0-BL
- added C65: 100nF, PCM_JLCPCB:C_0603, F.Cu at (209.5, 58.2)
- added C_sense7: 100nF, PCM_JLCPCB:C_0603, F.Cu at (106.8, 49.4)
- added C_sense8: 100nF, PCM_JLCPCB:C_0603, F.Cu at (106.8, 51.6)
- added C_sense9: 100nF, PCM_JLCPCB:C_0603, F.Cu at (106.8, 53.9)
- added DSub1: DR-15P圆针公蓝色, easyeda2kicad:D-SUB-TH_BOOMELE_DR-15P, F.Cu at (169.5, 63.5)
- added DSub2: DS1038-15FBNSIA74-0CC, easyeda2kicad:DSUB-TH_DS1038-15FBNSIA74-0CC, F.Cu at (169.8, 41.0)
- added J5: 2.54-1*6PHeader-RA, easyeda2kicad:HDR-TH_6P-P2.54-H-M-W10.0, F.Cu at (205.7, 104.4)
- added Q14: 2N7002, easyeda2kicad:SOT-23-3_L2.9-W1.3-P1.90-LS2.4-BR, F.Cu at (208.4, 119.8)
- added Q17: CJQ4435, easyeda2kicad:SOP-8_L5.0-W4.0-P1.27-LS6.2-BL, F.Cu at (199.5, 115.1)
- added Q18: CJQ4435, easyeda2kicad:SOP-8_L5.0-W4.0-P1.27-LS6.2-BL, F.Cu at (216.3, 119.0)
- added Q21: 2N7002, easyeda2kicad:SOT-23-3_L2.9-W1.3-P1.90-LS2.4-BR, F.Cu at (198.2, 46.1)
- added Q22: CJQ4435, easyeda2kicad:SOP-8_L5.0-W4.0-P1.27-LS6.2-BL, F.Cu at (199.5, 39.8)
- added Q23: currentmirror, easyeda2kicad:SOT-363-6_L2.2-W1.3-P0.65-LS2.1-BL, F.Cu at (208.1, 123.6)
- added Q24: 2N7002, easyeda2kicad:SOT-23-3_L2.9-W1.3-P1.90-LS2.4-BR, F.Cu at (198.2, 50.3)
- added Q25: 2N7002, easyeda2kicad:SOT-23-3_L2.9-W1.3-P1.90-LS2.4-BR, F.Cu at (198.2, 54.5)
- added Q26: 2N7002, easyeda2kicad:SOT-23-3_L2.9-W1.3-P1.90-LS2.4-BR, F.Cu at (198.2, 58.7)
- added Q27: CJQ4435, easyeda2kicad:SOP-8_L5.0-W4.0-P1.27-LS6.2-BL, F.Cu at (206.2, 39.8)
- added Q28: CJQ4435, easyeda2kicad:SOP-8_L5.0-W4.0-P1.27-LS6.2-BL, F.Cu at (212.8, 39.8)
- added R68: RM065-204(200K), easyeda2kicad:RES-ADJ-TH_3P-L7.3-W6.4-P5.00-R, F.Cu at (211.4, 48.3)
- added RPROG10: 1kΩ, PCM_JLCPCB:R_0603, F.Cu at (205.8, 51.9)
- added RPROG11: 1kΩ, PCM_JLCPCB:R_0603, F.Cu at (227.4, 70.7)
- added RPROG12: 1kΩ, PCM_JLCPCB:R_0603, F.Cu at (227.4, 73.0)
- added RPROG13: 1kΩ, PCM_JLCPCB:R_0603, F.Cu at (227.4, 75.2)
- added RPROG14: 1kΩ, PCM_JLCPCB:R_0603, F.Cu at (227.4, 77.5)
- added RPROG15: 1kΩ, PCM_JLCPCB:R_0603, F.Cu at (227.4, 79.7)
- added RPROG8: 1kΩ, PCM_JLCPCB:R_0603, F.Cu at (204.5, 123.2)
- added RPROG9: 1kΩ, PCM_JLCPCB:R_0603, F.Cu at (205.8, 49.6)
- added R_sense5: 100Ω, PCM_JLCPCB:R_0603, F.Cu at (119.4, 40.4)
- added R_sense6: 100Ω, PCM_JLCPCB:R_0603, F.Cu at (119.4, 42.6)
- added R_sense7: 100Ω, PCM_JLCPCB:R_0603, F.Cu at (119.4, 44.9)
- added Rsense3: LTR18EZPFSR015, easyeda2kicad:R0612, F.Cu at (123.2, 34.8)
- added SW3: TS-1088R-02026, easyeda2kicad:SW-SMD_L3.9-W3.0-P4.45, F.Cu at (112.0, 52.3)
- added TP2: TestPoint, Connector_PinHeader_2.54mm:PinHeader_1x01_P2.54mm_Vertical, F.Cu at (133.8, 45.8)
- C10, C11: value 22uF -> 10uf; footprint PCM_JLCPCB:C_0603 -> easyeda2kicad:C0805
- C12: value 100nF -> 10uf; footprint PCM_JLCPCB:C_0603 -> easyeda2kicad:C0805
- C13: value 22uf -> 100nF; footprint easyeda2kicad:C1206 -> PCM_JLCPCB:C_0603
- C14, C22, C29: value 10uF -> 100nF
- C15: value 4.7uF -> 100nF
- C16: value 47nF -> 100nF
- C19, C3, C6: value 100nF -> 100nf; footprint PCM_JLCPCB:C_0603 -> easyeda2kicad:C0805
- C2: value 22uf -> 100nf
- C21: value 100nF -> 330uf; footprint PCM_JLCPCB:C_0603 -> easyeda2kicad:CAP-SMD_BD10.0-L10.3-W10.3-FD
- C23: value 4.7uF -> 470uf; footprint PCM_JLCPCB:C_0603 -> easyeda2kicad:CAP-SMD_BD10.0-L10.3-W10.3-LS11.0-FD
- C24, C25: value 330pF -> 470uf; footprint PCM_JLCPCB:C_0603 -> easyeda2kicad:CAP-SMD_BD10.0-L10.3-W10.3-LS11.0-FD
- C27: value 10uF -> 100nF; footprint PCM_JLCPCB:C_1206 -> PCM_JLCPCB:C_0805
- C35, C36: value 22uF -> 100nF
- C38: value 100nF -> 1uF
- C39: value 47pF -> 1uF
- C4: value 22uF -> 22uf; footprint PCM_JLCPCB:C_0603 -> easyeda2kicad:C0805
- C40: value 22uF -> 4.7uF
- C5: value 100nF -> 22uf; footprint PCM_JLCPCB:C_0603 -> easyeda2kicad:C0805
- C7: value 22uF -> 100nf; footprint PCM_JLCPCB:C_0603 -> easyeda2kicad:C0805
- C8: value 10uF -> 10uf; footprint PCM_JLCPCB:C_0603 -> easyeda2kicad:C0805
- D1: value 1N4148W -> SS54_C22452; footprint Diode_SMD:D_SOD-123 -> easyeda2kicad:SMA_L4.4-W2.8-LS5.4-R-RD
- D10: value Yellow -> Green
- D11: value H5VU10U -> 1N4148W; footprint PCM_JLCPCB:D_DFN1006-2L -> Diode_SMD:D_SOD-123
- D12: value MBR0530 -> Green; footprint easyeda2kicad:SOD-123_L2.8-W1.8-LS3.7-RD -> PCM_JLCPCB:D_0805
- D13, D3: value Green -> BZX84C5V6; footprint PCM_JLCPCB:D_0805 -> PCM_JLCPCB:D_SOT-23
- D14: value SS14 -> BZX84C3V3; footprint PCM_JLCPCB:D_SMA -> PCM_JLCPCB:D_SOT-23
- D2: value H5VU10U -> SS54_C22452; footprint PCM_JLCPCB:D_DFN1006-2L -> easyeda2kicad:SMA_L4.4-W2.8-LS5.4-R-RD
- D5: value SS34 -> SS54_C22452; footprint PCM_JLCPCB:D_SMA -> easyeda2kicad:SMA_L4.4-W2.8-LS5.4-R-RD
- D6: value SS34 -> BZX84C5V6; footprint PCM_JLCPCB:D_SMA -> PCM_JLCPCB:D_SOT-23
- D7: value Red -> BZX84C5V6; footprint PCM_JLCPCB:D_0805 -> PCM_JLCPCB:D_SOT-23
- L1: value 22uH -> SPM6530T-2R2M; footprint easyeda2kicad:IND-SMD_L7.5-W7.5 -> easyeda2kicad:IND-SMD_L7.1-W6.5-P5.60
- L3: value 22uH -> SMDRI127-330MT; footprint easyeda2kicad:IND-SMD_L7.5-W7.5 -> easyeda2kicad:IND-SMD_L12.3-W12.3
- L5: value 10uh -> SMDRI127-330MT; footprint easyeda2kicad:IND-SMD_L7.5-W6.6 -> easyeda2kicad:IND-SMD_L12.3-W12.3
- P10, P4, P5: value 1.27mm/1*3p -> Header-Male-2.54_1x1; footprint easyeda2kicad:HDR-TH_3P-P1.27-V-M-1 -> easyeda2kicad:HDR-TH_1P-P2.54-V-M
- P2: value Header-Male-2.54_2x2 -> Header-Male-2.54_1x1; footprint easyeda2kicad:HDR-TH_4P-P2.54-V-M-R2-C2-S2.54-1 -> easyeda2kicad:HDR-TH_1P-P2.54-V-M
- P3: value 1.27mm/1*3p -> Header-Male-2.54_2x2; footprint easyeda2kicad:HDR-TH_3P-P1.27-V-M-1 -> easyeda2kicad:HDR-TH_4P-P2.54-V-M-R2-C2-S2.54-1
- Q11: value AO3401A -> BSS84; footprint easyeda2kicad:SOT-23_L2.9-W1.3-P1.90-LS2.4-BR -> Package_TO_SOT_SMD:SOT-23
- R1: value 11.3kohm -> 0805W8F2553T5E; footprint easyeda2kicad:R1206 -> easyeda2kicad:R0805
- R10: value 22kΩ -> 1kΩ; footprint PCM_JLCPCB:R_0603 -> PCM_JLCPCB:R_0805
- R11, R26: value 1MΩ -> 10kΩ; footprint PCM_JLCPCB:R_0603 -> PCM_JLCPCB:R_0805
- R14: value 10kΩ -> 1MΩ; footprint PCM_JLCPCB:R_0603 -> PCM_JLCPCB:R_0805
- R16: footprint PCM_JLCPCB:R_0603 -> PCM_JLCPCB:R_0805
- R2: value 215kohm -> 0805W8F5102T5E; footprint easyeda2kicad:R0402 -> easyeda2kicad:R0805
- R21: value 5.1kΩ -> 1kΩ; footprint PCM_JLCPCB:R_0603 -> PCM_JLCPCB:R_0805
- R22: value 240Ω -> 1kΩ; footprint PCM_JLCPCB:R_0603 -> PCM_JLCPCB:R_0805
- R24: value 2.2kΩ -> 10kΩ; footprint PCM_JLCPCB:R_0603 -> PCM_JLCPCB:R_0805
- R25: value 150Ω -> 10kΩ; footprint PCM_JLCPCB:R_0603 -> PCM_JLCPCB:R_0805
- R3: value 3kΩ -> 0805W8F5102T5E; footprint PCM_JLCPCB:R_0603 -> easyeda2kicad:R0805
- R32: value 100Ω -> 5.1kΩ
- R33: value 10Ω -> 5.1kΩ
- R37: value 49.9kΩ -> 10kΩ
- R38, R50: value 100kΩ -> 10kΩ
- R4: value 10Ω -> 0.5ohm; footprint PCM_JLCPCB:R_0402 -> easyeda2kicad:R1206
- R40: value 511k -> 5.1kΩ; footprint easyeda2kicad:R0805 -> PCM_JLCPCB:R_0603
- R41, R43: value 105k -> 10kΩ; footprint easyeda2kicad:R0603 -> PCM_JLCPCB:R_0603
- R44: value 49.9kΩ -> 5.1kΩ
- R45: value 100kΩ -> 5.1kΩ
- R46: value 3kΩ -> 100kΩ
- R47: value 511k -> 10kΩ; footprint easyeda2kicad:R0805 -> PCM_JLCPCB:R_0603
- R48: value 105k -> 100kΩ; footprint easyeda2kicad:R0603 -> PCM_JLCPCB:R_0603
- R49: value 49.9kΩ -> 100kΩ
- R5: value 5.23k -> 100k
- R51: value 13.3k -> 100kΩ; footprint easyeda2kicad:R0805 -> PCM_JLCPCB:R_0603
- R52: value 22kΩ -> 1MΩ
- R53: value 2.2kΩ -> 1kΩ; footprint PCM_JLCPCB:R_0603 -> PCM_JLCPCB:R_0805
- R54: value RM065-204(200K) -> 1MΩ; footprint easyeda2kicad:RES-ADJ-TH_3P-L7.3-W6.4-P5.00-R -> PCM_JLCPCB:R_0603
- R6: value 100kΩ -> 4.7k; footprint PCM_JLCPCB:R_0603 -> easyeda2kicad:R0805
- R8: value 10kΩ -> 4.7k; footprint PCM_JLCPCB:R_0603 -> easyeda2kicad:R0805
- R9: value 10kΩ -> 1kΩ; footprint PCM_JLCPCB:R_0603 -> PCM_JLCPCB:R_0805
- U1: value MAX17048G+T10 -> IP2326; footprint easyeda2kicad:TDFN-8_L2.0-W2.0-P0.50-BL-EP1.2 -> easyeda2kicad:VQFN-24_L4.0-W4.0-P0.50-BL-EP2.5
- U10: value BQ25606RGER -> MAX3232CDBR; footprint easyeda2kicad:VQFN-24_L4.0-W4.0-P0.50-TL-EP2.8 -> easyeda2kicad:SSOP-16_L6.2-W5.3-P0.65-LS7.8-BL
- U12: value BQ24170RGYR -> ADS1115IDGSR; footprint easyeda2kicad:VQFN-24_L5.5-W3.5-P0.50-BL-EP-2 -> easyeda2kicad:MSOP-10_L3.0-W3.0-P0.50-LS5.0-BL
- U19: value TPS54302DDCR_C311983 -> TPL5110DDCT; footprint easyeda2kicad:SOT-23-6_L2.9-W1.6-P0.95-LS2.8-BL -> easyeda2kicad:TSOT-23-6_L2.9-W1.6-P0.95-LS2.8-BR
- U2: value MT3608 -> MAX17048G+T10; footprint easyeda2kicad:SOT-23-6_L2.9-W1.6-P0.95-LS2.8-BL -> easyeda2kicad:TDFN-8_L2.0-W2.0-P0.50-BL-EP1.2
- U3: value MT3608 -> 90KR; footprint easyeda2kicad:SOT-23-6_L2.9-W1.6-P0.95-LS2.8-BL -> easyeda2kicad:R0805
- U4: value TPL5110DDCT -> LM2596SX-3.3; footprint easyeda2kicad:TSOT-23-6_L2.9-W1.6-P0.95-LS2.8-BR -> easyeda2kicad:TO-263-5_L10.2-W8.6-P1.70-LS14.4-TL
- U6: value MT3608 -> LM2596SX-5.0/NOPB; footprint PCM_JLCPCB:SOT-23-6_L2.9-W1.6-P0.95-LS2.8-BL -> easyeda2kicad:TO-263-5_L10.2-W8.9-P1.70-TL
- U7: value Z-21320110021001 -> 2.54-2*20; footprint easyeda2kicad:HDR-TH_20P-P2.54-V-M-R2-C10-S2.54 -> easyeda2kicad:HDR-TH_40P-P2.54-V-F-R2-C20-S2.54
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Connections:
- C10 pad 1: /3V3VSYS -> /3S IC/BAT+
- C10 pad 2: /3V3GND -> /GND
- C11 pad 1: /3V3GND -> /GND
- C11 pad 2: /3V3VOUT -> Net-(U1-VIN)
- C12 pad 1: /Temp3.3V -> /3S IC/ICVBUS
- C12 pad 2: /TEMPGND -> /GND
- C13 pad 1: Net-(U10-PMID) -> /DSUB+RS232/DSUB3.3V
- C13 pad 2: /GND1 -> /GND
- C14 pad 1: /GND1 -> /3S Balancer/VC5
- C14 pad 2: /VBAT1 -> /3S Balancer/VC3
- C15 pad 1: /REGN1 -> /3S Balancer/VC3
- C15 pad 2: /GND1 -> /3S Balancer/VC1
- C16 pad 1: Net-(U10-BTST) -> /3S Balancer/VC1
- C16 pad 2: Net-(C16-Pad2) -> /3S Balancer/GND
- C18 pad 1: Net-(U8-V+) -> /3S Balancer/GND
- C18 pad 2: /DSUBGND -> /3S Balancer/VC0
- C19 pad 1: Net-(U8-C2+) -> /DSUB+RS232/DSUB3.3V
- C19 pad 2: Net-(U8-C2-) -> /GND
- C2 pad 1: /12GND -> Net-(U1-BST)
- C2 pad 2: /12VSYS -> Net-(C2-Pad2)
- C21 pad 1: /DSUB3.3V -> /5V
- C21 pad 2: /DSUBGND -> /GND
- C22 pad 1: /GND1 -> Net-(U10-C1+)
- C22 pad 2: /VSYS1 -> Net-(U10-C1-)
- C23 pad 1: /VCC -> /LM2596 BUCK/LM2596_VIN
- C23 pad 2: /BAT_3 (-) -> /GND
- C24 pad 1: /CC2 -> /DSUB+RS232/DSUB3.3V
- C24 pad 2: /PDGND -> /GND
- C25 pad 1: /CC1 -> /LM2596 BUCK/LM2596_VIN
- C25 pad 2: /PDGND -> /GND
- C27 pad 1: Net-(Q7-D) -> /3S Balancer/TS1
- C27 pad 2: /PDGND -> /3S Balancer/GND
- C29 pad 1: /3V3BVSYS -> Net-(U10-V+)
- C29 pad 2: /3V3BGND -> /GND
- C3 pad 1: /SLEEPSIG -> /LM2596 BUCK/LM2596_VIN
- C3 pad 2: /SLEEPGND -> /GND
- C33 pad 1: Net-(U13-BOOT) -> /DSUB+RS232/DSUB3.3V
- C33 pad 2: /3V3BOOT -> /GND
- C35 pad 1: /12BVOUT -> Net-(U10-V-)
- C35 pad 2: /12BGND -> /GND
- C36 pad 1: /12BVOUT -> Net-(U10-C2+)
- C36 pad 2: /12BGND -> Net-(U10-C2-)
- C38 pad 1: /12BVSYS -> /3S IC/BAT+
- C38 pad 2: /12BGND -> /3S Balancer/GND
- C39 pad 1: Net-(C39-Pad1) -> Net-(U8-CAP1)
- C39 pad 2: /3V3FB -> Net-(U8-VSS)
- C4 pad 1: /5GND -> /GND
- C4 pad 2: /5VOUT -> /Load Sharing/VSYS
- C40 pad 1: /3V3BVOUT -> Net-(U8-REGOUT)
- C40 pad 2: /3V3BGND -> /3S Balancer/GND
- C5 pad 1: Net-(Q10-D) -> /GND
- C5 pad 2: Net-(Q11-S) -> /Load Sharing/VSYS
- C6 pad 1: Net-(Q11-S) -> /GND
- C6 pad 2: /CHG_GND -> /LM2596 BUCK/LM2596_VIN
- C7 pad 1: /5VSYS -> /GND
- C7 pad 2: /5GND -> /5V
- C8 pad 1: /BAT_3 (-) -> /3S IC/BAT+
- C8 pad 2: Net-(U15-BAT) -> /GND
- D1 pad 1: Net-(D1-K) -> /Load Sharing/VSYS
- D1 pad 2: Net-(D1-A) -> /LM2596 BUCK/LM2596_VIN
- D10 pad 1: Net-(D10-Pad1) -> /GND
- D10 pad 2: /V1VSYS -> Net-(D10-Pad2)
- D11 pad 1: /CC2 -> Net-(D11-K)
- D11 pad 2: /PDGND -> Net-(D11-A)
- D12 pad 1: Net-(D100-C) -> /GND
- D12 pad 2: /12V_Adapter -> Net-(D12-Pad2)
- D13 pad 1: Net-(U12-STAT) -> /3S Balancer/VC1
- D13 pad 2: Net-(D13-Pad2) -> (no net)
- D14 pad 1: /VBUS1 -> /3S Balancer/GND
- D14 pad 2: /GND1 -> (no net)
- D2 pad 1: /CC1 -> /GND
- D2 pad 2: /PDGND -> /LM2596 5V Buck/SW
- D3 pad 1: Net-(D3-Pad1) -> /3S Balancer/B3-
- D3 pad 2: /V1VSYS -> (no net)
- D5 pad 1: /5VOUT -> /GND
- D5 pad 2: Net-(U2-SW) -> /LM2596 BUCK/SW
- D6 pad 1: /3V3VOUT -> /3S Balancer/B1+
- D6 pad 2: Net-(U6-SW) -> (no net)
- D7 pad 1: Net-(D7-Pad1) -> /3S Balancer/B1-
- D7 pad 2: /V1VSYS -> (no net)
- D8 pad 1: Net-(D8-Pad1) -> /GND
- D8 pad 2: /VSYS1 -> Net-(D8-Pad2)
- D9 pad 1: Net-(D9-Pad1) -> /GND
- D9 pad 2: /VSYS1 -> Net-(D9-Pad2)
- L1 pad 1: /5VSYS -> Net-(C2-Pad2)
- L1 pad 2: Net-(U2-SW) -> /3S IC/ICVBUS
- L3 pad 1: /3V3VSYS -> /LM2596 5V Buck/SW
- L3 pad 2: Net-(U6-SW) -> /5V
- L5 pad 1: /5BOOT -> /LM2596 BUCK/SW
- L5 pad 2: /5BVOUT -> /DSUB+RS232/DSUB3.3V
- P10 pad 1: /V1VBUS -> /DSUB+RS232/DSUB12V
- P2 pad 1: /FUELSDA -> /GPIO14/TXD0
- P3 pad 1: /SLEEPVSYS -> /GPIO2/SDA1
- P3 pad 2: /SLEEPGND -> /3S IC/BAT+
- P3 pad 3: /SLEEPSIG -> /GPIO3/SCL1
- P4 pad 1: /3V3BVSYS -> /GPIO15/RXD0
- P5 pad 1: /12VSYS -> /DSUB+RS232/DSUB3.3V
- Q11 pad 1: Net-(Q11-G) -> /3S Balancer/GND
- Q11 pad 2: Net-(Q11-S) -> /3S Balancer/CHG
- Q11 pad 3: /CHG_VBAT -> Net-(D11-A)
- Q5 pad 1: /PROTECT- -> /3S Balancer/PROTECT-
- Q5 pad 2: Net-(Q5A-G1) -> /3S Balancer/DSG
- Q5 pad 4: Net-(D1-K) -> Net-(D11-K)
- Q5 pad 5: /PACK- -> /GND
- Q5 pad 6: /PACK- -> /GND
- R1 pad 1: /12GND -> /TEMP+HEATER/base
- R1 pad 2: Net-(U3-FB) -> /DSUB+RS232/DSUB3.3V
- R10 pad 1: /5VOUT -> /3S Balancer/B3-
- R10 pad 2: Net-(U2-FB) -> /3S Balancer/VC3
- R11 pad 1: Net-(Q5A-G1) -> Net-(Q3-G)
- R11 pad 2: /PROTECT- -> /3S Balancer/VC3
- R14 pad 1: Net-(Q1-D) -> Net-(U8-ALERT)
- R14 pad 2: /TEMP12V -> /3S Balancer/GND
- R15 pad 1: Net-(D1-A) -> /3S Balancer/DSG
- R15 pad 2: Net-(D1-K) -> /3S Balancer/PROTECT-
- R16 pad 1: Net-(R16-Pad1) -> Net-(Q9-G)
- R16 pad 2: Net-(U15-TS1) -> /3S Balancer/VC1
- R2 pad 1: /12VOUT -> /GND
- R2 pad 2: Net-(U3-FB) -> Net-(U1-NTC)
- R21 pad 1: /Temp3.3V -> /3S Balancer/B1+
- R21 pad 2: /TEMPSDA -> /3S Balancer/VC1
- R22 pad 1: /GND1 -> /3S Balancer/ALERT
- R22 pad 2: Net-(U10-ICHG) -> Net-(U8-ALERT)
- R24 pad 1: Net-(D9-Pad1) -> Net-(Q10-G)
- R24 pad 2: Net-(U10-~{PG}) -> /3S Balancer/VC0
- R25 pad 1: /GND1 -> /3S Balancer/TS1
- R25 pad 2: Net-(U10-ILIM) -> /3S Balancer/GND
- R26 pad 1: Net-(D1-K) -> Net-(R26-Pad1)
- R26 pad 2: /PACK- -> /3S Balancer/TS1
- R3 pad 1: Net-(U2-FB) -> /3S IC/ICVBUS
- R3 pad 2: /5GND -> /3S IC/ICEN
- R31 pad 1: Net-(USBC1-CC1) -> /GND
- R31 pad 2: /USBGND -> Net-(USBC1-CC2)
- R32 pad 1: /BAT_1 (+) -> /GND
- R32 pad 2: Net-(U15-BAT) -> Net-(USBC1-CC1)
- R33 pad 1: Net-(Q7-D) -> /GND
- R33 pad 2: Net-(U17-VIN) -> /3S IC/ICVBUS
- R37 pad 1: /12BVOUT -> /SLEEPMOSFET/SLPSIG
- R37 pad 2: Net-(C49-Pad1) -> /GND
- R38 pad 1: Net-(C49-Pad1) -> /SLEEPMOSFET/SLPDRV
- R38 pad 2: /12FB -> /GND
- R39 pad 2: /V1GND -> /DSUB+RS232/DSUB12V
- R4 pad 1: Net-(D100-C) -> Net-(U1-VIN)
- R4 pad 2: Net-(U12-AVCC) -> /3S IC/ICVBUS
- R40 pad 1: Net-(U19-EN) -> /DSUB+RS232/DSUB3.3V
- R40 pad 2: /12BVSYS -> Net-(U12-ALERT/RDY)
- R41 pad 1: /12BGND -> /GND
- R41 pad 2: Net-(U19-EN) -> /GPIO23
- R43 pad 1: /3V3BGND -> Net-(Q21-D)
- R43 pad 2: Net-(U13-EN) -> /DSUB+RS232/DSUB3.3V
- R44 pad 1: /3V3BVOUT -> /DSUB+RS232/DSUB3.3V
- R44 pad 2: Net-(C39-Pad1) -> /GPIO2/SDA1
- R45 pad 1: Net-(C39-Pad1) -> /DSUB+RS232/DSUB3.3V
- R45 pad 2: /3V3FB -> /GPIO3/SCL1
- R46 pad 1: /12BGND -> /DSUB+RS232/DSUB3.3V
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Routing:
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- removed copper zone on F.Cu, net /12GND
- removed copper zone on F.Cu, net /3V3GND
- removed copper zone on F.Cu, net /5GND
Other:
- board outline removed
- board text removed: "12V"
- board text removed: "3V3"
- board text removed: "3v3"
- board text removed: "5V"
- board text removed: "ADDR"
- board text removed: "B1+"
- board text removed: "B1-"
- board text removed: "B1- B2+"
- board text removed: "B2-"
- board text removed: "B2- B3+"
- board text removed: "B3- GND"
- board text removed: "BAT"
- board text removed: "BTST"
- board text removed: "CE"
- board text removed: "CHG_GND"
- board text removed: "CHG_VBAT"
- board text removed: "D+"
- board text removed: "D-"
- board text removed: "GND"
- board text removed: "ICHG"
- board text removed: "ILIM"
- board text removed: "ISET"
- board text removed: "OTG"
- board text removed: "PG"
- board text removed: "PMID"
- board text removed: "REGN"
- board text removed: "RX"
- board text removed: "RX_13V"
- board text removed: "SCL"
- board text removed: "SDA"
- board text removed: "SIG"
- board text removed: "STAT"
- board text removed: "SW"
- board text removed: "SYS"
- board text removed: "TS"
- board text removed: "TX"
- board text removed: "TX_13V"
- board text removed: "V+"
- board text removed: "V-"
- board text removed: "VAC"
- board text removed: "VBAT"
- board text removed: "VBUS"
- board text removed: "VOUT"
- board text removed: "VSET"
- board text removed: "VSYS"

Commit message: sunday
Parts:
- removed DSub1: DR-15P圆针公蓝色, easyeda2kicad:D-SUB-TH_BOOMELE_DR-15P
- removed J5: 2.54-1*6PHeader-RA, easyeda2kicad:HDR-TH_6P-P2.54-H-M-W10.0
- removed P10, P2, P4, P5: Header-Male-2.54_1x1, easyeda2kicad:HDR-TH_1P-P2.54-V-M
- removed P3: Header-Male-2.54_2x2, easyeda2kicad:HDR-TH_4P-P2.54-V-M-R2-C2-S2.54-1
- removed R68: RM065-204(200K), easyeda2kicad:RES-ADJ-TH_3P-L7.3-W6.4-P5.00-R
- added ? (x2): , , F.Cu at (80.1, 71.9)
- added ? (x2): , , F.Cu at (103.1, 130.0)
- added ?: , , F.Cu at (80.1, 130.0)
- added ? (x4): , , F.Cu at (103.1, 71.9)
- added CN1: DC3-2.54-14PAL, easyeda2kicad:IDC-TH_14P-P2.54_ZHOURI_DC3-2.54-14PAL, F.Cu at (121.3, 91.2)
- added Q1: DMN2004K-7, easyeda2kicad:SOT-23-3_L3.0-W1.7-P0.95-LS2.9-BR, B.Cu at (90.0, 144.1)
- added Q2: DMN2004K-7, easyeda2kicad:SOT-23-3_L3.0-W1.7-P0.95-LS2.9-BR, B.Cu at (96.7, 143.6)
- added Q3: DMN2004K-7, easyeda2kicad:SOT-23-3_L3.0-W1.7-P0.95-LS2.9-BR, B.Cu at (100.5, 146.1)
- added R12: 62kΩ, PCM_JLCPCB:R_0805, F.Cu at (95.9, 172.1)
- added R13: 33Ω, PCM_JLCPCB:R_0805, B.Cu at (99.5, 149.2)
- added R18: 51kΩ, PCM_JLCPCB:R_0805, F.Cu at (88.3, 167.5)
- added R19: 51kΩ, PCM_JLCPCB:R_0805, F.Cu at (97.8, 172.1)
- added R20: 33Ω, PCM_JLCPCB:R_0805, B.Cu at (96.0, 141.1)
- added TP10: VSYS, Connector_PinHeader_2.54mm:PinHeader_1x01_P2.54mm_Vertical, F.Cu at (96.0, 130.0)
- added TP15: SDA, Connector_PinHeader_2.54mm:PinHeader_1x01_P2.54mm_Vertical, F.Cu at (76.3, 140.3)
- added TP16: SCL, Connector_PinHeader_2.54mm:PinHeader_1x01_P2.54mm_Vertical, F.Cu at (76.3, 135.8)
- added TP3: TestPoint, Connector_PinHeader_2.54mm:PinHeader_1x01_P2.54mm_Vertical, B.Cu at (96.5, 138.1)
- added TP4: TestPoint, Connector_PinHeader_2.54mm:PinHeader_1x01_P2.54mm_Vertical, B.Cu at (92.5, 138.1)
- added TP5: TestPoint, Connector_PinHeader_2.54mm:PinHeader_1x01_P2.54mm_Vertical, B.Cu at (88.5, 138.1)
- added TP6: BAT-, Connector_PinHeader_2.54mm:PinHeader_1x01_P2.54mm_Vertical, F.Cu at (76.3, 162.2)
- added TP7: Bat+, Connector_PinHeader_2.54mm:PinHeader_1x01_P2.54mm_Vertical, F.Cu at (76.3, 158.5)
- added TP8: VBUS, Connector_PinHeader_2.54mm:PinHeader_1x01_P2.54mm_Vertical, F.Cu at (76.3, 154.9)
- added TP9: TestPoint, Connector_PinHeader_2.54mm:PinHeader_1x01_P2.54mm_Vertical, F.Cu at (76.3, 151.3)
- C14, C15, C16, C18, C27, C38, C39, C40, C65, C_sense7, C_sense8, C_sense9, D1, D11, D13, D14, D3, D6, D7, Q11, Q18, Q21, Q22, Q24, Q25, Q26, Q27, Q28, Q5, R10, R11, R14, R15, R16, R21, R22, R24, R25, R26, R37, R38, R41, R43, R46, R47, R48, R49, R5, R52, R53, R54, R9, RPROG10, RPROG9, R_sense5, R_sense6, R_sense7, Rsense3, SW3, TP2, U19, U2: moved to B.Cu
- R2, R3: value 0805W8F5102T5E -> 4.7kΩ; footprint easyeda2kicad:R0805 -> PCM_JLCPCB:R_0805
- R6: value 4.7k -> 3362P-1-204; footprint easyeda2kicad:R0805 -> easyeda2kicad:RES-ADJ-TH_3P-L7.1-W6.9-P2.50-L_3362P
- R8: value 4.7k -> 33Ω; footprint easyeda2kicad:R0805 -> PCM_JLCPCB:R_0805; moved to B.Cu
- U3: value 90KR -> BQ7692003PWR; footprint easyeda2kicad:R0805 -> easyeda2kicad:TSSOP-20_L6.5-W4.4-P0.65-LS6.4-BL; moved to B.Cu
- moved USBC1 184.5 mm to (81.0, 168.8)
- moved R32 176.9 mm to (79.7, 163.7), turned to -90 degrees
- moved D8 176.7 mm to (90.3, 167.4), turned to 90 degrees
- moved R31 175.7 mm to (82.7, 163.7), turned to -90 degrees
- moved D9 173.9 mm to (92.5, 168.8), turned to -90 degrees
- moved U3 171.3 mm to (95.0, 157.5)
- moved R6 168.5 mm to (116.3, 167.6), turned to 90 degrees
- moved RPROG11 167.6 mm to (94.1, 172.4), turned to -90 degrees
- moved U1 166.8 mm to (97.3, 166.7), turned to -90 degrees
- moved RPROG14 166.2 mm to (90.1, 171.2), turned to 180 degrees
- moved RPROG12 164.0 mm to (94.2, 168.7), turned to -90 degrees
- moved RPROG15 163.5 mm to (92.4, 172.1), turned to -90 degrees
- moved RPROG13 162.5 mm to (92.9, 166.5), turned to 180 degrees
- moved R3 161.0 mm to (92.1, 125.2)
- moved C2 160.0 mm to (101.8, 168.7), turned to -90 degrees
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Connections:
- net /LM2596 BUCK/LM2596_VIN renamed /LM2596 3V3 BUCK/LM2596_VIN
- net /LM2596 BUCK/SW renamed /LM2596 3V3 BUCK/SW
- C10 pad 2: /GND -> /3S IC/ICGND
- C11 pad 1: /GND -> /3S IC/ICGND
- C12 pad 2: /GND -> /3S IC/ICGND
- C39 pad 1: Net-(U8-CAP1) -> Net-(U3-VC0)
- C39 pad 2: Net-(U8-VSS) -> Net-(U3-VC4)
- C4 pad 1: /GND -> /3S IC/ICGND
- C40 pad 1: Net-(U8-REGOUT) -> Net-(U3-SRP)
- C5 pad 1: /GND -> /3S IC/ICGND
- C8 pad 2: /GND -> /3S IC/ICGND
- D6 pad 1: /3S Balancer/B1+ -> /FUELGAUGE/FUELBAT
- D8 pad 1: /GND -> /3S IC/ICGND
- D9 pad 1: /GND -> /3S IC/ICGND
- Q5 pad 5: /GND -> /3S IC/ICGND
- Q5 pad 6: /GND -> /3S IC/ICGND
- R14 pad 1: Net-(U8-ALERT) -> Net-(U3-BAT)
- R2 pad 1: /GND -> /5V
- R2 pad 2: Net-(U1-NTC) -> Net-(D10-Pad2)
- R21 pad 1: /3S Balancer/B1+ -> /FUELGAUGE/FUELBAT
- R22 pad 1: /3S Balancer/ALERT -> /GPIO25
- R22 pad 2: Net-(U8-ALERT) -> Net-(U3-BAT)
- R3 pad 1: /3S IC/ICVBUS -> /DSUB+RS232/DSUB3.3V
- R3 pad 2: /3S IC/ICEN -> Net-(D12-Pad2)
- R31 pad 1: /GND -> /3S IC/ICGND
- R32 pad 1: /GND -> /3S IC/ICGND
- R33 pad 1: /GND -> /3S IC/ICGND
- R54 pad 2: /GND -> /3S IC/ICGND
- R6 pad 1: Net-(D10-Pad2) -> unconnected-(R6-Pad1)
- R6 pad 2: /5V -> /GND
- R8 pad 1: Net-(D12-Pad2) -> /3S IC/BAT+
- R8 pad 2: /DSUB+RS232/DSUB3.3V -> Net-(Q1-D)
- RPROG11 pad 2: /GND -> /3S IC/ICGND
- RPROG14 pad 2: /GND -> /3S IC/ICGND
- RPROG15 pad 2: /GND -> /3S IC/ICGND
- R_sense7 pad 2: Net-(U8-BAT) -> Net-(U3-ALERT)
- U1 pad 18: /GND -> /3S IC/ICGND
- U1 pad 25: /GND -> /3S IC/ICGND
- U2 pad 2: /3S IC/BAT+ -> /FUELGAUGE/FUELBAT
- U3 pad 1: Net-(U1-ISET) -> unconnected-(U3-DSG-Pad1)
- U3 pad 2: /GND -> /3S Balancer/VC5
- U7 pad 1: /raspi3.3V -> /5V
- U7 pad 10: /GPIO15/RXD0 -> /GND
- U7 pad 11: /GPIO17 -> /GPIO18/PCM.CLK
- U7 pad 12: /GPIO18/PCM.CLK -> /GPIO17
- U7 pad 13: /GPIO27 -> /GND
- U7 pad 14: /GND -> /GPIO27
- U7 pad 15: /GPIO22 -> /GPIO23
- U7 pad 16: /GPIO23 -> /GPIO22
- U7 pad 17: /raspi3.3V -> /GPIO24
- U7 pad 18: /GPIO24 -> /raspi3.3V
- U7 pad 19: /GPIO10/SPI0.MOSI -> /GND
- U7 pad 2: /5V -> /raspi3.3V
- U7 pad 20: /GND -> /GPIO10/SPI0.MOSI
- U7 pad 21: /GPIO9/SPI0.MISO -> /GPIO25
- U7 pad 22: /GPIO25 -> /GPIO9/SPI0.MISO
- U7 pad 23: /GPIO11/SPI0.SCLK -> /GPIO8/SPI0.CE0
- U7 pad 24: /GPIO8/SPI0.CE0 -> /GPIO11/SPI0.SCLK
- U7 pad 25: /GND -> /GPIO7/SPI0.CE1
- U7 pad 26: /GPIO7/SPI0.CE1 -> /GND
- U7 pad 27: /ID_SDA -> /ID_SCL
- U7 pad 28: /ID_SCL -> /ID_SDA
- U7 pad 29: /GPIO5 -> /GND
- U7 pad 3: /GPIO2/SDA1 -> /5V
- U7 pad 30: /GND -> /GPIO5
- U7 pad 31: /GPIO6 -> /GPIO12/PWM0
- U7 pad 32: /GPIO12/PWM0 -> /GPIO6
- U7 pad 33: /GPIO13/PWM1 -> /GND
- U7 pad 34: /GND -> /GPIO13/PWM1
- U7 pad 35: /GPIO19/PCM.FS -> /GPIO16
- U7 pad 36: /GPIO16 -> /GPIO19/PCM.FS
- U7 pad 37: /GPIO26 -> /GPIO20/PCM.DIN
- U7 pad 38: /GPIO20/PCM.DIN -> /GPIO26
- U7 pad 39: /GND -> /GPIO21/PCM.DOUT
- U7 pad 4: /5V -> /GPIO2/SDA1
- U7 pad 40: /GPIO21/PCM.DOUT -> /GND
- U7 pad 5: /GPIO3/SCL1 -> /GND
- U7 pad 6: /GND -> /GPIO3/SCL1
- U7 pad 7: /GPIO4/GPCLK0 -> /GPIO14/TXD0
- U7 pad 8: /GPIO14/TXD0 -> /GPIO4/GPCLK0
- U7 pad 9: /GND -> /GPIO15/RXD0
- USBC1 pad 1: /GND -> /3S IC/ICGND
- USBC1 pad 2: /GND -> /3S IC/ICGND
- USBC1 pad 3: /GND -> /3S IC/ICGND
- USBC1 pad 4: /GND -> /3S IC/ICGND
- USBC1 pad A1B12: /GND -> /3S IC/ICGND
- USBC1 pad B1A12: /GND -> /3S IC/ICGND
Routing:
- net /3S IC/BAT+: track 0.00 -> 85.2 mm, vias 0 -> 2
- net /3S IC/ICVBUS: track 0.00 -> 65.9 mm, vias 0 -> 3
- net /3S IC/ICEN: track 0.00 -> 45.2 mm
- net /LM2596 3V3 BUCK/LM2596_VIN: track 0.00 -> 36.4 mm
- net /DSUB+RS232/DSUB3.3V: track 0.00 -> 36.2 mm, vias 0 -> 1
- net /3S Balancer/VC1: track 0.00 -> 29.2 mm
- net /SLEEPMOSFET/SLPDRV: track 0.00 -> 28.5 mm, vias 0 -> 3
- net /3S Balancer/VC0: track 0.00 -> 23.8 mm
- net /3S IC/DP: track 0.00 -> 22.3 mm
- net /FUELGAUGE/FUELBAT: track 0.00 -> 21.0 mm
- net /3S IC/DN: track 0.00 -> 19.6 mm
- net /SLEEPMOSFET/SLPSIG: track 0.00 -> 18.5 mm
- net /SLEEPMOSFET/5EN: track 0.00 -> 18.3 mm, vias 0 -> 1
- net /3S Balancer/B3-: track 0.00 -> 15.7 mm
- net /3S Balancer/PROTECT-: track 0.00 -> 15.5 mm
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Other:
- board outline added: 60 x 126.9 mm

Commit message: Voltage Regulators Wired
Parts:
- moved L3 73.0 mm to (90.7, 78.5), turned to 90 degrees
- moved D10 70.1 mm to (89.3, 97.8)
- moved C7 69.9 mm to (97.7, 96.3), turned to 180 degrees
- moved R2 65.9 mm to (92.8, 97.8), turned to 180 degrees
- moved C21 61.5 mm to (90.2, 91.3), turned to 180 degrees
- moved U6 57.4 mm to (106.7, 78.9)
- moved C6 55.1 mm to (111.7, 85.3), turned to 180 degrees
- moved D2 51.1 mm to (109.7, 90.5), turned to -90 degrees
- moved R51 48.2 mm to (112.2, 73.8), turned to 180 degrees
- moved C25 46.5 mm to (102.7, 89.8), turned to -90 degrees
- moved TP5 40.0 mm to (105.9, 174.1), turned to 0 degrees
- moved TP4 37.2 mm to (101.9, 174.1), turned to 0 degrees
- moved TP2 36.6 mm to (93.9, 174.1), turned to 0 degrees
- moved TP3 36.1 mm to (97.9, 174.1), turned to 0 degrees
- moved C19 34.9 mm to (114.3, 103.7), turned to 90 degrees
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Routing:
- net /DSUB+RS232/DSUB3.3V: track 36.2 -> 101.4 mm
- net /5V: track 0.00 -> 65.0 mm
- net /LM2596 5V Buck/SW: track 0.00 -> 33.0 mm
- net /LM2596 3V3 BUCK/SW: track 0.00 -> 28.2 mm
- net /LM2596 3V3 BUCK/LM2596_VIN: track 36.4 -> 59.6 mm
- net /SLEEPMOSFET/5EN: track 18.3 -> 20.5 mm
- net Net-(D10-Pad2): track 0.00 -> 1.65 mm

Commit message: Finished Everything Except For Ground and USBC Errors
Parts:
- added ?: , , F.Cu at (78.0, 132.0)
- added ?: , , F.Cu at (108.6, 132.0)
- added ?: , , F.Cu at (88.2, 132.0)
- added ?: , , F.Cu at (118.7, 132.0)
- added ?: , , F.Cu at (98.4, 132.0)
- C13, C22, C29, C33, C35, C36, Q14, Q17, Q23, R1, R39, R40, R44, R45, R50, RPROG8, U10, U12: moved to B.Cu
- U2: moved to F.Cu
- moved RPROG10 37.7 mm to (101.5, 134.5), turned to -90 degrees
- moved U12 37.2 mm to (102.0, 90.9), turned to -90 degrees
- moved Q14 36.2 mm to (95.0, 82.4), turned to -90 degrees
- moved Q27 35.7 mm to (98.0, 136.5), turned to 180 degrees
- moved R37 35.5 mm to (115.0, 138.5), turned to 90 degrees
- moved R44 35.3 mm to (97.5, 89.9)
- moved Q26 34.7 mm to (105.0, 136.5), turned to -90 degrees
- moved RPROG9 34.6 mm to (113.5, 138.5), turned to 90 degrees
- moved Q25 33.9 mm to (93.5, 139.5), turned to 180 degrees
- moved C65 33.8 mm to (112.0, 138.5), turned to 90 degrees
- moved R39 33.5 mm to (97.5, 82.2), turned to -90 degrees
- moved R45 33.3 mm to (97.5, 88.7)
- moved Q24 33.3 mm to (109.0, 138.0), turned to 90 degrees
- moved R50 32.8 mm to (95.1, 84.9), turned to 180 degrees
- moved R48 31.4 mm to (101.5, 139.0), turned to 90 degrees
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Routing:
- net /GPIO2/SDA1: track 0.00 -> 128.0 mm, vias 0 -> 6
- net /GPIO3/SCL1: track 0.00 -> 127.7 mm, vias 0 -> 7
- net /DSUB+RS232/DSUB12V: track 11.4 -> 114.9 mm, vias 1 -> 6
- net /DSUB+RS232/DSUB3.3V: track 101.4 -> 191.2 mm, vias 1 -> 3
- net /GPIO25: track 0.00 -> 82.3 mm, vias 0 -> 4
- net /LM2596 3V3 BUCK/LM2596_VIN: track 59.6 -> 122.7 mm, vias 0 -> 3
- net /GPIO23: track 14.6 -> 76.1 mm
- net /SLEEPMOSFET/5EN: track 20.5 -> 75.9 mm
- net /TEMP+HEATER/HEATER+: track 0.00 -> 40.6 mm
- net /FUELGAUGE/FUELBAT: track 21.0 -> 60.3 mm
- net /3S Balancer/CHG: track 8.60 -> 45.1 mm, vias 2 -> 4
- net /GPIO18/PCM.CLK: track 0.00 -> 24.9 mm, vias 0 -> 3
- net /raspi3.3V: track 0.00 -> 24.7 mm
- net /GND: track 0.00 -> 23.3 mm, vias 0 -> 4
- net /GPIO15/RXD0: track 0.00 -> 21.7 mm
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- added copper zone on B.Cu, net /GND
- added copper zone on F.Cu, net /GND
Other:
- board size 60 x 126.9 mm -> 48.8 x 127.4 mm

Commit message: finished
Parts:
- removed the ? at (88.2, 132.0)
- removed the ? at (118.7, 132.0)
- removed the ? at (98.4, 132.0)
- added ?: , , F.Cu at (118.5, 132.0)
- added ?: , , F.Cu at (98.0, 132.0)
- added ?: , , F.Cu at (88.0, 132.0)
- added TP17: 12VOUT, Connector_PinHeader_2.54mm:PinHeader_1x01_P2.54mm_Vertical, F.Cu at (119.0, 68.5)
- added TP18: 3V3, Connector_PinHeader_2.54mm:PinHeader_1x01_P2.54mm_Vertical, F.Cu at (119.0, 73.1)
- added TP19: TX, Connector_PinHeader_2.54mm:PinHeader_1x01_P2.54mm_Vertical, F.Cu at (76.5, 61.0)
- added TP20: RX, Connector_PinHeader_2.54mm:PinHeader_1x01_P2.54mm_Vertical, F.Cu at (76.5, 56.0)
- added TP21: 5V, Connector_PinHeader_2.54mm:PinHeader_1x01_P2.54mm_Vertical, F.Cu at (77.0, 65.5)
- R54: moved to F.Cu
- moved TP15 14.8 mm to (81.5, 126.0), turned to -90 degrees
- moved TP16 13.4 mm to (85.5, 126.0), turned to -90 degrees
- moved R5 6.66 mm to (94.0, 151.5), turned to -90 degrees
- moved Q21 5.52 mm to (109.9, 141.4)
- moved R6 5.52 mm to (115.9, 149.7)
- moved C65 5.52 mm to (117.4, 139.5)
- moved Q22 5.52 mm to (117.4, 143.5)
- moved Q24 5.52 mm to (114.4, 139.0)
- moved Q25 5.52 mm to (98.9, 140.5)
- moved Q26 5.52 mm to (110.4, 137.5)
- moved Q27 5.52 mm to (103.4, 137.5)
- moved Q28 5.52 mm to (104.4, 145.5)
- moved R37 5.52 mm to (120.4, 139.5)
- moved R38 5.52 mm to (97.9, 143.5)
- moved R41 5.52 mm to (108.9, 144.0)
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Connections:
- C10 pad 2: /3S IC/ICGND -> /GND
- C11 pad 1: /3S IC/ICGND -> /GND
- C12 pad 2: /3S IC/ICGND -> /GND
- C16 pad 2: /3S Balancer/GND -> /GND
- C18 pad 1: /3S Balancer/GND -> /GND
- C27 pad 2: /3S Balancer/GND -> /GND
- C38 pad 2: /3S Balancer/GND -> /GND
- C39 pad 1: Net-(U3-VC0) -> Net-(U3-CAP1)
- C39 pad 2: Net-(U3-VC4) -> Net-(U3-VSS)
- C4 pad 1: /3S IC/ICGND -> /GND
- C40 pad 1: Net-(U3-SRP) -> Net-(U3-REGOUT)
- C40 pad 2: /3S Balancer/GND -> /GND
- C5 pad 1: /3S IC/ICGND -> /GND
- C8 pad 2: /3S IC/ICGND -> /GND
- C_sense7 pad 1: /3S Balancer/GND -> /GND
- C_sense9 pad 2: /3S Balancer/GND -> /GND
- D14 pad 1: /3S Balancer/GND -> /GND
- D8 pad 1: /3S IC/ICGND -> /GND
- D9 pad 1: /3S IC/ICGND -> /GND
- Q11 pad 1: /3S Balancer/GND -> /GND
- Q5 pad 5: /3S IC/ICGND -> /GND
- Q5 pad 6: /3S IC/ICGND -> /GND
- R12 pad 1: /3S IC/ICGND -> /GND
- R14 pad 1: Net-(U3-BAT) -> Net-(U3-ALERT)
- R14 pad 2: /3S Balancer/GND -> /GND
- R18 pad 1: /3S IC/ICGND -> /GND
- R22 pad 2: Net-(U3-BAT) -> Net-(U3-ALERT)
- R25 pad 2: /3S Balancer/GND -> /GND
- R31 pad 1: /3S IC/ICGND -> /GND
- R32 pad 1: /3S IC/ICGND -> /GND
- R33 pad 1: /3S IC/ICGND -> /GND
- R54 pad 2: /3S IC/ICGND -> /GND
- RPROG11 pad 2: /3S IC/ICGND -> /GND
- RPROG14 pad 2: /3S IC/ICGND -> /GND
- RPROG15 pad 2: /3S IC/ICGND -> /GND
- R_sense6 pad 2: /3S Balancer/GND -> /GND
- R_sense7 pad 2: Net-(U3-ALERT) -> Net-(U3-BAT)
- Rsense3 pad 2: /3S Balancer/GND -> /GND
- TP6 pad 1: /3S IC/ICGND -> /GND
- U1 pad 18: /3S IC/ICGND -> /GND
- U1 pad 25: /3S IC/ICGND -> /GND
- U3 pad 1: unconnected-(U3-DSG-Pad1) -> /3S Balancer/DSG
- U3 pad 11: /3S Balancer/DSG -> unconnected-(U3-NC-Pad11)
- U3 pad 12: /3S Balancer/CHG -> /3S Balancer/VC5
- U3 pad 13: Net-(U3-VC4) -> /3S Balancer/VC3
- U3 pad 14: /GPIO2/SDA1 -> /3S Balancer/VC3
- U3 pad 15: /GPIO3/SCL1 -> /3S Balancer/VC3
- U3 pad 16: /3S Balancer/TS1 -> /3S Balancer/VC1
- U3 pad 17: Net-(U3-VC0) -> /3S Balancer/VC0
- U3 pad 18: Net-(U3-SRP) -> /3S Balancer/SRP
- U3 pad 19: /3S IC/BAT+ -> /3S Balancer/SRN
- U3 pad 2: /3S Balancer/VC5 -> /3S Balancer/CHG
- U3 pad 3: /3S Balancer/VC3 -> Net-(U3-VSS)
- U3 pad 4: /3S Balancer/VC3 -> /GPIO2/SDA1
- U3 pad 5: /3S Balancer/VC3 -> /GPIO3/SCL1
- U3 pad 6: /3S Balancer/VC1 -> /3S Balancer/TS1
- U3 pad 7: /3S Balancer/VC0 -> Net-(U3-CAP1)
- U3 pad 8: /3S Balancer/SRP -> Net-(U3-REGOUT)
- U3 pad 9: /3S Balancer/SRN -> /3S IC/BAT+
- USBC1 pad 1: /3S IC/ICGND -> /GND
- USBC1 pad 2: /3S IC/ICGND -> /GND
- USBC1 pad 3: /3S IC/ICGND -> /GND
- USBC1 pad 4: /3S IC/ICGND -> /GND
- USBC1 pad A1B12: /3S IC/ICGND -> /GND
- USBC1 pad B1A12: /3S IC/ICGND -> /GND
Routing:
- net /GND: track 23.3 -> 226.6 mm, vias 4 -> 28
- net /GPIO15/RXD0: track 21.7 -> 55.3 mm
- net /DSUB+RS232/DSUB3.3V: track 191.2 -> 215.6 mm, vias 3 -> 5
- net /DSUB+RS232/DSUB12V: track 114.9 -> 136.3 mm
- net /GPIO14/TXD0: track 20.6 -> 41.3 mm
- net /3S IC/ICGND: track 18.1 -> 0.00 mm
- net /LM2596 3V3 BUCK/LM2596_VIN: track 122.7 -> 131.6 mm
- net /5V: track 77.8 -> 85.3 mm
- net /3S Balancer/VC0: track 23.8 -> 30.3 mm
- net /GPIO2/SDA1: track 128.0 -> 132.6 mm, vias 6 -> 4
- net Net-(Q3-G): track 8.31 -> 12.6 mm
- net Net-(U3-SRP): track 4.15 -> 0.00 mm
- net Net-(U3-REGOUT): track 0.00 -> 4.15 mm
- net Net-(U3-VSS): track 0.00 -> 2.70 mm
- net Net-(U3-VC4): track 2.70 -> 0.00 mm
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Other:
- board size 48.8 x 127.4 mm -> 49.8 x 126.5 mm

Commit message: tuesday
Parts:
- removed the ? at (-53.5, 51.0)
- added TP11: VSYS2, Connector_PinHeader_2.54mm:PinHeader_1x01_P2.54mm_Vertical, F.Cu at (103.0, 125.0)
- added TP23: GND, Connector_PinHeader_2.54mm:PinHeader_1x01_P2.54mm_Vertical, F.Cu at (118.5, 110.3)
- added TP24: GND, Connector_PinHeader_2.54mm:PinHeader_1x01_P2.54mm_Vertical, F.Cu at (118.5, 114.9)
- added TP25: GND, Connector_PinHeader_2.54mm:PinHeader_1x01_P2.54mm_Vertical, F.Cu at (118.5, 119.5)
Connections:
- DSub2 pad 1: /DSUB+RS232/UART_RX_13V -> /GPIO15/RXD0
- DSub2 pad 2: /DSUB+RS232/UART_TX_13V -> /GPIO14/TXD0
- U10 pad 13: /DSUB+RS232/UART_RX_13V -> /GPIO15/RXD0
- U10 pad 14: /DSUB+RS232/UART_TX_13V -> /GPIO14/TXD0
Routing:
- net /GPIO14/TXD0: track 41.3 -> 75.2 mm, vias 0 -> 2
- net /DSUB+RS232/UART_RX_13V: track 15.9 -> 0.00 mm
- net /DSUB+RS232/UART_TX_13V: track 15.9 -> 0.00 mm
- net /GPIO15/RXD0: track 55.3 -> 57.2 mm

Commit message: labeled
Parts:
- moved TP2 0.54 mm to (117.0, 167.5)
- moved TP5 0.54 mm to (117.0, 155.5)
- renumbered TP17 to 12V, TP18 to 3V3, TP24 to GND, TP25 to GND, TP23 to GND, TP20 to RX, TP19 to TX, TP11 to VSYS
Routing:
- net /FUELGAUGE/FUELBAT: track 60.3 -> 60.8 mm
- net /3S Balancer/B3-: track 14.5 -> 15.0 mm
- net /3S Balancer/B1-: track 9.36 -> 9.91 mm
Other:
- board text added: "3S BALANCER"
- board text added: "3V3"
- board text added: "5V"
- board text added: "B+"
- board text added: "B-"
- board text added: "B1+"
- board text added: "B1-"
- board text added: "B3+"
- board text added: "B3-"
- board text added: "ICEN"
- board text added: "SCL"
- board text added: "SDA"
- board text added: "SLEEP TIMER"
- board text added: "TEMP+HEAT"
- board text added: "VBUS"
- board text added: "VSENS"
- board text added: "VSYS"
